File: kicad/pbx-sniffer/pbx-sniffer.kicad_pcb (KiCad board)
At the start: 2 copper layers, 319 parts, among them K10 Relay_SPDT, K11 Relay_SPST-NO, K12 Relay_SPDT, K13 Relay_SPST-NO, K14 Relay_SPDT, K15 Relay_SPST-NO, K16 Relay_SPDT, K17 Relay_SPST-NO, K18 Relay_SPDT, K19 Relay_SPST-NO, K2 Relay_SPST-NO, K20 Relay_SPDT, K21 Relay_SPST-NO, K22 Relay_SPDT, K23 Relay_SPST-NO, K24 Relay_SPDT, K25 Relay_SPST-NO, K26 Relay_SPDT, K27 Relay_SPST-NO, K28 Relay_SPDT, K29 Relay_SPST-NO, K3 Relay_SPDT, K30 Relay_SPDT, K31 Relay_SPST-NO, K32 Relay_SPDT, K33 Relay_SPST-NO, K34 Relay_SPDT, K35 Relay_SPST-NO, K36 Relay_SPDT, K37 Relay_SPST-NO, K38 Relay_SPDT, K39 Relay_SPST-NO, K40 Relay_SPDT, K41 Relay_SPST-NO, K42 Relay_SPDT, K43 Relay_SPST-NO, K44 Relay_SPDT, K45 Relay_SPST-NO, K46 Relay_SPDT, K47 Relay_SPST-NO, K48 Relay_SPDT, K49 Relay_SPST-NO, K5 Relay_SPST-NO, K50 Relay_SPDT, K6 Relay_SPDT, K7 Relay_SPST-NO, K8 Relay_SPDT, K9 Relay_SPST-NO, Q10 PMOS, Q11 PMOS, Q12 PMOS, Q13 PMOS, Q14 PMOS, Q15 PMOS, Q16 PMOS, Q17 PMOS, Q18 PMOS, Q19 PMOS, Q2 PMOS, Q20 PMOS, Q21 PMOS, Q22 PMOS, Q23 PMOS, Q24 PMOS, Q25 PMOS, Q26 PMOS, Q27 PMOS, Q28 PMOS, Q29 PMOS, Q30 PMOS, Q31 PMOS, Q32 PMOS, Q33 PMOS, Q34 PMOS, Q35 PMOS, Q36 PMOS, Q37 PMOS, Q38 PMOS, Q39 PMOS, Q4 PMOS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

Commit message: begin organizing the pcb components for layout
Parts:
- moved J25 461.9 mm to (369.2, 302.0)
- moved J29 461.9 mm to (429.0, 302.0)
- moved J30 461.9 mm to (443.9, 302.0)
- moved J31 461.9 mm to (369.2, 324.8)
- moved J35 461.9 mm to (429.0, 324.8)
- moved J36 461.9 mm to (443.9, 324.8)
- moved J37 461.9 mm to (369.2, 347.7)
- moved J41 461.9 mm to (429.0, 347.7)
- moved J42 461.9 mm to (443.9, 347.7)
- moved J43 461.9 mm to (369.2, 370.5)
- moved J47 461.9 mm to (429.0, 370.5)
- moved J48 461.9 mm to (443.9, 370.5)
- moved J26 461.9 mm to (384.1, 302.0)
- moved J27 461.9 mm to (399.1, 302.0)
- moved J28 461.9 mm to (414.0, 302.0)
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Other:
- board text added: "Input Jacks"
- board text added: "Output Jacks"

Commit message: commenced placement on pcb
Parts:
- added JP10: JUP_P10mm, PCM_SL_Jumpers:JUP_P10mm, F.Cu at (140.0, 131.8)
- added JP11: JUP_P10mm, PCM_SL_Jumpers:JUP_P10mm, F.Cu at (406.0, 272.2)
- added JP12: JUP_P10mm, PCM_SL_Jumpers:JUP_P10mm, F.Cu at (406.0, 236.8)
- added JP13: JUP_P10mm, PCM_SL_Jumpers:JUP_P10mm, F.Cu at (375.9, 272.2)
- added JP14: JUP_P10mm, PCM_SL_Jumpers:JUP_P10mm, F.Cu at (375.9, 257.1)
- added JP15: JUP_P10mm, PCM_SL_Jumpers:JUP_P10mm, F.Cu at (375.9, 262.1)
- added JP16: JUP_P10mm, PCM_SL_Jumpers:JUP_P10mm, F.Cu at (390.9, 272.2)
- added JP17: JUP_P10mm, PCM_SL_Jumpers:JUP_P10mm, F.Cu at (406.0, 267.1)
- added JP18: JUP_P10mm, PCM_SL_Jumpers:JUP_P10mm, F.Cu at (142.4, 117.6)
- added JP19: JUP_P10mm, PCM_SL_Jumpers:JUP_P10mm, F.Cu at (390.9, 252.0)
- added JP2: JUP_P10mm, PCM_SL_Jumpers:JUP_P10mm, F.Cu at (139.0, 146.8)
- added JP20: JUP_P10mm, PCM_SL_Jumpers:JUP_P10mm, F.Cu at (375.9, 241.9)
- added JP21: JUP_P10mm, PCM_SL_Jumpers:JUP_P10mm, F.Cu at (390.9, 236.8)
- added JP22: JUP_P10mm, PCM_SL_Jumpers:JUP_P10mm, F.Cu at (406.0, 252.0)
- added JP23: JUP_P10mm, PCM_SL_Jumpers:JUP_P10mm, F.Cu at (390.9, 267.1)
- added JP24: JUP_P10mm, PCM_SL_Jumpers:JUP_P10mm, F.Cu at (375.9, 267.1)
- added JP25: JUP_P10mm, PCM_SL_Jumpers:JUP_P10mm, F.Cu at (406.0, 262.1)
- added JP3: JUP_P10mm, PCM_SL_Jumpers:JUP_P10mm, F.Cu at (375.9, 236.8)
- added JP4: JUP_P10mm, PCM_SL_Jumpers:JUP_P10mm, F.Cu at (390.9, 257.1)
- added JP5: JUP_P10mm, PCM_SL_Jumpers:JUP_P10mm, F.Cu at (406.0, 246.9)
- added JP6: JUP_P10mm, PCM_SL_Jumpers:JUP_P10mm, F.Cu at (406.0, 257.1)
- added JP7: JUP_P10mm, PCM_SL_Jumpers:JUP_P10mm, F.Cu at (406.0, 241.9)
- added JP8: JUP_P10mm, PCM_SL_Jumpers:JUP_P10mm, F.Cu at (390.9, 262.1)
- added JP9: JUP_P10mm, PCM_SL_Jumpers:JUP_P10mm, F.Cu at (375.9, 252.0)
- K11, K13, K15, K17, K19, K21, K23, K25, K27, K29, K31, K33, K35, K37, K39, K41, K43, K45, K47, K49, K5, K7, K9: footprint Relay_THT:Relay_StandexMeder_DIP_HighProfile -> Relay_THT:Relay_SPST_StandexMeder_SIL_Form1A
- K3: renamed from K2; footprint Relay_THT:Relay_StandexMeder_DIP_HighProfile -> Relay_THT:Relay_SPST_StandexMeder_SIL_Form1A
- moved U9 497.0 mm to (23.5, 213.2), turned to 90 degrees
- moved U4 488.8 mm to (25.6, 231.4)
- moved U5 488.8 mm to (36.4, 231.4)
- moved U6 488.8 mm to (47.2, 231.4)
- moved U8 481.4 mm to (23.7, 195.0), turned to 90 degrees
- moved U7 466.1 mm to (23.9, 176.1), turned to 90 degrees
- moved J41 416.4 mm to (147.6, 40.8), turned to 180 degrees
- moved J1 385.4 mm to (649.1, -2.77)
- moved R86 379.0 mm to (129.3, 127.4), turned to 180 degrees
- moved U18 371.7 mm to (137.0, 133.1), turned to 180 degrees
- moved R78 366.6 mm to (128.2, 143.2), turned to 180 degrees
- moved U10 359.8 mm to (135.6, 148.9), turned to 180 degrees
- moved U1 347.5 mm to (14.2, 88.3)
- moved R94 345.8 mm to (131.8, 112.8), turned to 180 degrees
- moved J31 340.6 mm to (147.7, 66.0), turned to 180 degrees
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- renumbered D2 to D4, D3 to D5, D4 to D6, D5 to D7, D6 to D8, J7 to J1, J4 to J10, J5 to J11, J6 to J12, J8 to J2, J9 to J3, J10 to J4, J11 to J5, J12 to J6, J1 to J7, J2 to J8, J3 to J9, K3 to K4, Q2 to Q3, R2 to R6, R3 to R7, R4 to R8, U4 to U10, U5 to U4, U6 to U5, U7 to U6, U8 to U7, U9 to U8, U10 to U9
Connections:
- D4 pad 1: Net-(D2-K) -> Net-(D4-K)
- D5 pad 1: Net-(D3-K) -> Net-(D5-K)
- D6 pad 1: Net-(D4-K) -> Net-(D6-K)
- D7 pad 1: Net-(D5-K) -> Net-(D7-K)
- D8 pad 1: Net-(D6-K) -> Net-(D8-K)
- K10 pad 1: (no net) -> Net-(D11-K)
- K10 pad 2: (no net) -> /Input Phone Jacks/Line Control3/Tpbx
- K10 pad 4: (no net) -> unconnected-(K10-Pad4)
- K10 pad 6: (no net) -> /Input Phone Jacks/Tpbx3
- K10 pad 8: (no net) -> GNDD
- K11 pad 1: (no net) -> Net-(K11-Pad1)
- K11 pad 7: (no net) -> /Input Phone Jacks/Rpbx4
- K12 pad 1: (no net) -> Net-(D13-K)
- K12 pad 2: (no net) -> /Input Phone Jacks/Line Control4/Tpbx
- K12 pad 4: (no net) -> unconnected-(K12-Pad4)
- K12 pad 6: (no net) -> /Input Phone Jacks/Tpbx4
- K12 pad 8: (no net) -> GNDD
- K13 pad 1: (no net) -> Net-(K13-Pad1)
- K13 pad 7: (no net) -> /Input Phone Jacks/Rpbx5
- K14 pad 1: (no net) -> Net-(D15-K)
- K14 pad 2: (no net) -> /Input Phone Jacks/Line Control5/Tpbx
- K14 pad 4: (no net) -> unconnected-(K14-Pad4)
- K14 pad 6: (no net) -> /Input Phone Jacks/Tpbx5
- K14 pad 8: (no net) -> GNDD
- K15 pad 1: (no net) -> Net-(K15-Pad1)
- K15 pad 7: (no net) -> /Input Phone Jacks/Rpbx6
- K16 pad 1: (no net) -> Net-(D17-K)
- K16 pad 2: (no net) -> /Input Phone Jacks/Line Control6/Tpbx
- K16 pad 4: (no net) -> unconnected-(K16-Pad4)
- K16 pad 6: (no net) -> /Input Phone Jacks/Tpbx6
- K16 pad 8: (no net) -> GNDD
- K17 pad 1: (no net) -> Net-(K17-Pad1)
- K17 pad 7: (no net) -> /Input Phone Jacks/Rpbx7
- K18 pad 1: (no net) -> Net-(D19-K)
- K18 pad 2: (no net) -> /Input Phone Jacks/Line Control7/Tpbx
- K18 pad 4: (no net) -> unconnected-(K18-Pad4)
- K18 pad 6: (no net) -> /Input Phone Jacks/Tpbx7
- K18 pad 8: (no net) -> GNDD
- K19 pad 1: (no net) -> Net-(K19-Pad1)
- K19 pad 7: (no net) -> /Input Phone Jacks/Rpbx8
- K20 pad 1: (no net) -> Net-(D21-K)
- K20 pad 2: (no net) -> /Input Phone Jacks/Line Control8/Tpbx
- K20 pad 4: (no net) -> unconnected-(K20-Pad4)
- K20 pad 6: (no net) -> /Input Phone Jacks/Tpbx8
- K20 pad 8: (no net) -> GNDD
- K21 pad 1: (no net) -> Net-(K21-Pad1)
- K21 pad 7: (no net) -> /Input Phone Jacks/Rpbx9
- K22 pad 1: (no net) -> Net-(D23-K)
- K22 pad 2: (no net) -> /Input Phone Jacks/Line Control9/Tpbx
- K22 pad 4: (no net) -> unconnected-(K22-Pad4)
- K22 pad 6: (no net) -> /Input Phone Jacks/Tpbx9
- K22 pad 8: (no net) -> GNDD
- K23 pad 1: (no net) -> Net-(K23-Pad1)
- K23 pad 7: (no net) -> /Input Phone Jacks/Rpbx10
- K24 pad 1: (no net) -> Net-(D25-K)
- K24 pad 2: (no net) -> /Input Phone Jacks/Line Control10/Tpbx
- K24 pad 4: (no net) -> unconnected-(K24-Pad4)
- K24 pad 6: (no net) -> /Input Phone Jacks/Tpbx10
- K24 pad 8: (no net) -> GNDD
- K25 pad 1: (no net) -> Net-(K25-Pad1)
- K25 pad 7: (no net) -> /Input Phone Jacks/Rpbx11
- K26 pad 1: (no net) -> Net-(D27-K)
- K26 pad 2: (no net) -> /Input Phone Jacks/Line Control11/Tpbx
- K26 pad 4: (no net) -> unconnected-(K26-Pad4)
- K26 pad 6: (no net) -> /Input Phone Jacks/Tpbx11
- K26 pad 8: (no net) -> GNDD
- K27 pad 1: (no net) -> Net-(K27-Pad1)
- K27 pad 7: (no net) -> /Input Phone Jacks/Rpbx12
- K28 pad 1: (no net) -> Net-(D29-K)
- K28 pad 2: (no net) -> /Input Phone Jacks/Line Control12/Tpbx
- K28 pad 4: (no net) -> unconnected-(K28-Pad4)
- K28 pad 6: (no net) -> /Input Phone Jacks/Tpbx12
- K28 pad 8: (no net) -> GNDD
- K29 pad 1: (no net) -> Net-(K29-Pad1)
- K29 pad 7: (no net) -> /Input Phone Jacks/Rpbx13
- K3 pad 1: (no net) -> Net-(K3-Pad1)
- K3 pad 7: (no net) -> /Input Phone Jacks/Rpbx0
- K30 pad 1: (no net) -> Net-(D31-K)
- K30 pad 2: (no net) -> /Input Phone Jacks/Line Control13/Tpbx
- K30 pad 4: (no net) -> unconnected-(K30-Pad4)
- K30 pad 6: (no net) -> /Input Phone Jacks/Tpbx13
- K30 pad 8: (no net) -> GNDD
- K31 pad 1: (no net) -> Net-(K31-Pad1)
- K31 pad 7: (no net) -> /Input Phone Jacks/Rpbx14
- K32 pad 1: (no net) -> Net-(D33-K)
- K32 pad 2: (no net) -> /Input Phone Jacks/Line Control14/Tpbx
- K32 pad 4: (no net) -> unconnected-(K32-Pad4)
- K32 pad 6: (no net) -> /Input Phone Jacks/Tpbx14
- K32 pad 8: (no net) -> GNDD
- K33 pad 1: (no net) -> Net-(K33-Pad1)
- K33 pad 7: (no net) -> /Input Phone Jacks/Rpbx15
- K34 pad 1: (no net) -> Net-(D35-K)
- K34 pad 2: (no net) -> /Input Phone Jacks/Line Control15/Tpbx
- K34 pad 4: (no net) -> unconnected-(K34-Pad4)
- K34 pad 6: (no net) -> /Input Phone Jacks/Tpbx15
- K34 pad 8: (no net) -> GNDD
- K35 pad 1: (no net) -> Net-(K35-Pad1)
- K35 pad 7: (no net) -> /Input Phone Jacks/Rpbx16
- K36 pad 1: (no net) -> Net-(D37-K)
- K36 pad 2: (no net) -> /Input Phone Jacks/Line Control16/Tpbx
- K36 pad 4: (no net) -> unconnected-(K36-Pad4)
- K36 pad 6: (no net) -> /Input Phone Jacks/Tpbx16
- K36 pad 8: (no net) -> GNDD
- K37 pad 1: (no net) -> Net-(K37-Pad1)
- K37 pad 7: (no net) -> /Input Phone Jacks/Rpbx17
- K38 pad 1: (no net) -> Net-(D39-K)
- K38 pad 2: (no net) -> /Input Phone Jacks/Line Control17/Tpbx
- K38 pad 4: (no net) -> unconnected-(K38-Pad4)
- K38 pad 6: (no net) -> /Input Phone Jacks/Tpbx17
- K38 pad 8: (no net) -> GNDD
- K39 pad 1: (no net) -> Net-(K39-Pad1)
- K39 pad 7: (no net) -> /Input Phone Jacks/Rpbx18
- K4 pad 1: (no net) -> Net-(D5-K)
- K4 pad 2: (no net) -> /Input Phone Jacks/Line Control0/Tpbx
- K4 pad 4: (no net) -> unconnected-(K4-Pad4)
- K4 pad 6: (no net) -> /Input Phone Jacks/Tpbx0
- K4 pad 8: (no net) -> GNDD
- K40 pad 1: (no net) -> Net-(D41-K)
- K40 pad 2: (no net) -> /Input Phone Jacks/Line Control18/Tpbx
- K40 pad 4: (no net) -> unconnected-(K40-Pad4)
- K40 pad 6: (no net) -> /Input Phone Jacks/Tpbx18
- K40 pad 8: (no net) -> GNDD
- K41 pad 1: (no net) -> Net-(K41-Pad1)
- K41 pad 7: (no net) -> /Input Phone Jacks/Rpbx19
- K42 pad 1: (no net) -> Net-(D43-K)
- K42 pad 2: (no net) -> /Input Phone Jacks/Line Control19/Tpbx
- K42 pad 4: (no net) -> unconnected-(K42-Pad4)
- K42 pad 6: (no net) -> /Input Phone Jacks/Tpbx19
- K42 pad 8: (no net) -> GNDD
- K43 pad 1: (no net) -> Net-(K43-Pad1)
- K43 pad 7: (no net) -> /Input Phone Jacks/Rpbx20
- K44 pad 1: (no net) -> Net-(D45-K)
- K44 pad 2: (no net) -> /Input Phone Jacks/Line Control20/Tpbx
- K44 pad 4: (no net) -> unconnected-(K44-Pad4)
- K44 pad 6: (no net) -> /Input Phone Jacks/Tpbx20
- K44 pad 8: (no net) -> GNDD
- K45 pad 1: (no net) -> Net-(K45-Pad1)
- K45 pad 7: (no net) -> /Input Phone Jacks/Rpbx21
- K46 pad 1: (no net) -> Net-(D47-K)
- K46 pad 2: (no net) -> /Input Phone Jacks/Line Control21/Tpbx
- K46 pad 4: (no net) -> unconnected-(K46-Pad4)
- K46 pad 6: (no net) -> /Input Phone Jacks/Tpbx21
- K46 pad 8: (no net) -> GNDD
- K47 pad 1: (no net) -> Net-(K47-Pad1)
- K47 pad 7: (no net) -> /Input Phone Jacks/Rpbx22
- K48 pad 1: (no net) -> Net-(D49-K)
- K48 pad 2: (no net) -> /Input Phone Jacks/Line Control22/Tpbx
- K48 pad 4: (no net) -> unconnected-(K48-Pad4)
- K48 pad 6: (no net) -> /Input Phone Jacks/Tpbx22
- K48 pad 8: (no net) -> GNDD
- K49 pad 1: (no net) -> Net-(K49-Pad1)
- K49 pad 7: (no net) -> /Input Phone Jacks/Rpbx23
- K5 pad 1: (no net) -> Net-(K5-Pad1)
- K5 pad 7: (no net) -> /Input Phone Jacks/Rpbx1
- K50 pad 1: (no net) -> Net-(D51-K)
- K50 pad 2: (no net) -> /Input Phone Jacks/Line Control23/Tpbx
- K50 pad 4: (no net) -> unconnected-(K50-Pad4)
- K50 pad 6: (no net) -> /Input Phone Jacks/Tpbx23
- K50 pad 8: (no net) -> GNDD
- K6 pad 1: (no net) -> Net-(D7-K)
- K6 pad 2: (no net) -> /Input Phone Jacks/Line Control1/Tpbx
- K6 pad 4: (no net) -> unconnected-(K6-Pad4)
- K6 pad 6: (no net) -> /Input Phone Jacks/Tpbx1
- K6 pad 8: (no net) -> GNDD
- K7 pad 1: (no net) -> Net-(K7-Pad1)
- K7 pad 7: (no net) -> /Input Phone Jacks/Rpbx2
- K8 pad 1: (no net) -> Net-(D9-K)
- K8 pad 2: (no net) -> /Input Phone Jacks/Line Control2/Tpbx
- K8 pad 4: (no net) -> unconnected-(K8-Pad4)
- K8 pad 6: (no net) -> /Input Phone Jacks/Tpbx2
- K8 pad 8: (no net) -> GNDD
- K9 pad 1: (no net) -> Net-(K9-Pad1)
- K9 pad 7: (no net) -> /Input Phone Jacks/Rpbx3
- Q3 pad 1: Net-(D2-K) -> Net-(D4-K)
- Q4 pad 1: Net-(D3-K) -> Net-(D5-K)
- Q5 pad 1: Net-(D4-K) -> Net-(D6-K)
- Q6 pad 1: Net-(D5-K) -> Net-(D7-K)
- Q7 pad 1: Net-(D6-K) -> Net-(D8-K)
- R10 pad 2: Net-(K5-Pad13) -> Net-(K5-Pad1)
- R13 pad 2: Net-(K7-Pad13) -> Net-(K7-Pad1)
- R16 pad 2: Net-(K9-Pad13) -> Net-(K9-Pad1)
- R19 pad 2: Net-(K11-Pad13) -> Net-(K11-Pad1)
- R22 pad 2: Net-(K13-Pad13) -> Net-(K13-Pad1)
- R25 pad 2: Net-(K15-Pad13) -> Net-(K15-Pad1)
- R28 pad 2: Net-(K17-Pad13) -> Net-(K17-Pad1)
- R31 pad 2: Net-(K19-Pad13) -> Net-(K19-Pad1)
- R34 pad 2: Net-(K21-Pad13) -> Net-(K21-Pad1)
- R37 pad 2: Net-(K23-Pad13) -> Net-(K23-Pad1)
- R40 pad 2: Net-(K25-Pad13) -> Net-(K25-Pad1)
- R43 pad 2: Net-(K27-Pad13) -> Net-(K27-Pad1)
- R46 pad 2: Net-(K29-Pad13) -> Net-(K29-Pad1)
- R49 pad 2: Net-(K31-Pad13) -> Net-(K31-Pad1)
- R52 pad 2: Net-(K33-Pad13) -> Net-(K33-Pad1)
- R55 pad 2: Net-(K35-Pad13) -> Net-(K35-Pad1)
- R58 pad 2: Net-(K37-Pad13) -> Net-(K37-Pad1)
- R61 pad 2: Net-(K39-Pad13) -> Net-(K39-Pad1)
- R64 pad 2: Net-(K41-Pad13) -> Net-(K41-Pad1)
- R67 pad 2: Net-(K43-Pad13) -> Net-(K43-Pad1)
- R7 pad 2: Net-(K2-Pad13) -> Net-(K3-Pad1)
- R70 pad 2: Net-(K45-Pad13) -> Net-(K45-Pad1)
- R73 pad 2: Net-(K47-Pad13) -> Net-(K47-Pad1)
- R76 pad 2: Net-(K49-Pad13) -> Net-(K49-Pad1)
- U1 pad 19: controlSW2 -> GND
- U1 pad 20: unconnected-(U1A-GND-Pad20) -> GND
- U1 pad 22: controlSW4 -> GND
- U1 pad 32: controlSW23 -> GND
- U1 pad 33: controlSW14 -> VBAT
- U1 pad 39: unconnected-(U1C-GND-Pad39) -> GND
- U1 pad 40: unconnected-(U1C-GND-Pad40) -> GND
- U1 pad 8: unconnected-(U1A-GND-Pad8) -> GND
- U1 pad 9: unconnected-(U1A-NC-Pad9)_1 -> GND

Commit message: add SPDT relay footprint and update symbol for it
Parts:
- K10, K12, K14, K16, K18, K20, K22, K24, K26, K28, K30, K32, K34, K36, K38, K4, K40, K42, K44, K46, K48, K50, K6, K8: footprint Relay_THT:Relay_SPDT_Panasonic_JW1_FormC -> Phones:K_AZ943-1C_AMZ
- moved K36 18.4 mm to (158.5, 143.3)
Connections:
- K10 pad 1: Net-(D11-K) -> /Input Phone Jacks/Tpbx3
- K10 pad 2: /Input Phone Jacks/Line Control3/Tpbx -> Net-(D11-K)
- K10 pad 4: unconnected-(K10-Pad4) -> /Input Phone Jacks/Line Control3/Tpbx
- K12 pad 1: Net-(D13-K) -> /Input Phone Jacks/Tpbx4
- K12 pad 2: /Input Phone Jacks/Line Control4/Tpbx -> Net-(D13-K)
- K12 pad 4: unconnected-(K12-Pad4) -> /Input Phone Jacks/Line Control4/Tpbx
- K14 pad 1: Net-(D15-K) -> /Input Phone Jacks/Tpbx5
- K14 pad 2: /Input Phone Jacks/Line Control5/Tpbx -> Net-(D15-K)
- K14 pad 4: unconnected-(K14-Pad4) -> /Input Phone Jacks/Line Control5/Tpbx
- K16 pad 1: Net-(D17-K) -> /Input Phone Jacks/Tpbx6
- K16 pad 2: /Input Phone Jacks/Line Control6/Tpbx -> Net-(D17-K)
- K16 pad 4: unconnected-(K16-Pad4) -> /Input Phone Jacks/Line Control6/Tpbx
- K18 pad 1: Net-(D19-K) -> /Input Phone Jacks/Tpbx7
- K18 pad 2: /Input Phone Jacks/Line Control7/Tpbx -> Net-(D19-K)
- K18 pad 4: unconnected-(K18-Pad4) -> /Input Phone Jacks/Line Control7/Tpbx
- K20 pad 1: Net-(D21-K) -> /Input Phone Jacks/Tpbx8
- K20 pad 2: /Input Phone Jacks/Line Control8/Tpbx -> Net-(D21-K)
- K20 pad 4: unconnected-(K20-Pad4) -> /Input Phone Jacks/Line Control8/Tpbx
- K22 pad 1: Net-(D23-K) -> /Input Phone Jacks/Tpbx9
- K22 pad 2: /Input Phone Jacks/Line Control9/Tpbx -> Net-(D23-K)
- K22 pad 4: unconnected-(K22-Pad4) -> /Input Phone Jacks/Line Control9/Tpbx
- K24 pad 1: Net-(D25-K) -> /Input Phone Jacks/Tpbx10
- K24 pad 2: /Input Phone Jacks/Line Control10/Tpbx -> Net-(D25-K)
- K24 pad 4: unconnected-(K24-Pad4) -> /Input Phone Jacks/Line Control10/Tpbx
- K26 pad 1: Net-(D27-K) -> /Input Phone Jacks/Tpbx11
- K26 pad 2: /Input Phone Jacks/Line Control11/Tpbx -> Net-(D27-K)
- K26 pad 4: unconnected-(K26-Pad4) -> /Input Phone Jacks/Line Control11/Tpbx
- K28 pad 1: Net-(D29-K) -> /Input Phone Jacks/Tpbx12
- K28 pad 2: /Input Phone Jacks/Line Control12/Tpbx -> Net-(D29-K)
- K28 pad 4: unconnected-(K28-Pad4) -> /Input Phone Jacks/Line Control12/Tpbx
- K30 pad 1: Net-(D31-K) -> /Input Phone Jacks/Tpbx13
- K30 pad 2: /Input Phone Jacks/Line Control13/Tpbx -> Net-(D31-K)
- K30 pad 4: unconnected-(K30-Pad4) -> /Input Phone Jacks/Line Control13/Tpbx
- K32 pad 1: Net-(D33-K) -> /Input Phone Jacks/Tpbx14
- K32 pad 2: /Input Phone Jacks/Line Control14/Tpbx -> Net-(D33-K)
- K32 pad 4: unconnected-(K32-Pad4) -> /Input Phone Jacks/Line Control14/Tpbx
- K34 pad 1: Net-(D35-K) -> /Input Phone Jacks/Tpbx15
- K34 pad 2: /Input Phone Jacks/Line Control15/Tpbx -> Net-(D35-K)
- K34 pad 4: unconnected-(K34-Pad4) -> /Input Phone Jacks/Line Control15/Tpbx
- K36 pad 1: Net-(D37-K) -> /Input Phone Jacks/Tpbx16
- K36 pad 2: /Input Phone Jacks/Line Control16/Tpbx -> Net-(D37-K)
- K36 pad 4: unconnected-(K36-Pad4) -> /Input Phone Jacks/Line Control16/Tpbx
- K38 pad 1: Net-(D39-K) -> /Input Phone Jacks/Tpbx17
- K38 pad 2: /Input Phone Jacks/Line Control17/Tpbx -> Net-(D39-K)
- K38 pad 4: unconnected-(K38-Pad4) -> /Input Phone Jacks/Line Control17/Tpbx
- K4 pad 1: Net-(D5-K) -> /Input Phone Jacks/Tpbx0
- K4 pad 2: /Input Phone Jacks/Line Control0/Tpbx -> Net-(D5-K)
- K4 pad 4: unconnected-(K4-Pad4) -> /Input Phone Jacks/Line Control0/Tpbx
- K40 pad 1: Net-(D41-K) -> /Input Phone Jacks/Tpbx18
- K40 pad 2: /Input Phone Jacks/Line Control18/Tpbx -> Net-(D41-K)
- K40 pad 4: unconnected-(K40-Pad4) -> /Input Phone Jacks/Line Control18/Tpbx
- K42 pad 1: Net-(D43-K) -> /Input Phone Jacks/Tpbx19
- K42 pad 2: /Input Phone Jacks/Line Control19/Tpbx -> Net-(D43-K)
- K42 pad 4: unconnected-(K42-Pad4) -> /Input Phone Jacks/Line Control19/Tpbx
- K44 pad 1: Net-(D45-K) -> /Input Phone Jacks/Tpbx20
- K44 pad 2: /Input Phone Jacks/Line Control20/Tpbx -> Net-(D45-K)
- K44 pad 4: unconnected-(K44-Pad4) -> /Input Phone Jacks/Line Control20/Tpbx
- K46 pad 1: Net-(D47-K) -> /Input Phone Jacks/Tpbx21
- K46 pad 2: /Input Phone Jacks/Line Control21/Tpbx -> Net-(D47-K)
- K46 pad 4: unconnected-(K46-Pad4) -> /Input Phone Jacks/Line Control21/Tpbx
- K48 pad 1: Net-(D49-K) -> /Input Phone Jacks/Tpbx22
- K48 pad 2: /Input Phone Jacks/Line Control22/Tpbx -> Net-(D49-K)
- K48 pad 4: unconnected-(K48-Pad4) -> /Input Phone Jacks/Line Control22/Tpbx
- K50 pad 1: Net-(D51-K) -> /Input Phone Jacks/Tpbx23
- K50 pad 2: /Input Phone Jacks/Line Control23/Tpbx -> Net-(D51-K)
- K50 pad 4: unconnected-(K50-Pad4) -> /Input Phone Jacks/Line Control23/Tpbx
- K6 pad 1: Net-(D7-K) -> /Input Phone Jacks/Tpbx1
- K6 pad 2: /Input Phone Jacks/Line Control1/Tpbx -> Net-(D7-K)
- K6 pad 4: unconnected-(K6-Pad4) -> /Input Phone Jacks/Line Control1/Tpbx
- K8 pad 1: Net-(D9-K) -> /Input Phone Jacks/Tpbx2
- K8 pad 2: /Input Phone Jacks/Line Control2/Tpbx -> Net-(D9-K)
- K8 pad 4: unconnected-(K8-Pad4) -> /Input Phone Jacks/Line Control2/Tpbx

Commit message: fix nucleo footprint and update pin numbers
Connections:
- U1 pad 1: Cline0 -> unconnected-(U1A-PC10-Pad1)
- U1 pad 11: spi0clk -> unconnected-(U1A-NC-Pad11)
- U1 pad 12: spi0cs0 -> unconnected-(U1A-IOREF-Pad12)
- U1 pad 13: spi0miso -> unconnected-(U1A-PA13-Pad13)
- U1 pad 14: spi0cs1 -> unconnected-(U1A-RESET-Pad14)
- U1 pad 15: spi0mosi -> unconnected-(U1A-PA14-Pad15)
- U1 pad 17: controlSW0 -> unconnected-(U1A-PA15-Pad17)
- U1 pad 2: Cline1 -> unconnected-(U1A-PC11-Pad2)
- U1 pad 21: controlSW3 -> unconnected-(U1A-PB7-Pad21)
- U1 pad 23: controlSW5 -> unconnected-(U1A-PC13-Pad23)
- U1 pad 24: controlSW6 -> unconnected-(U1A-VIN-Pad24)
- U1 pad 25: controlSW7 -> unconnected-(U1A-PC14-Pad25)
- U1 pad 26: controlSW8 -> unconnected-(U1A-NC-Pad26)
- U1 pad 27: controlSW9 -> unconnected-(U1A-PC15-Pad27)
- U1 pad 28: controlSW10 -> unconnected-(U1A-PA0-Pad28)
- U1 pad 29: controlSW11 -> unconnected-(U1A-PF0-Pad29)
- U1 pad 3: Cline2 -> unconnected-(U1A-PC12-Pad3)
- U1 pad 30: controlSW12 -> unconnected-(U1A-PA1-Pad30)
- U1 pad 31: controlSW13 -> unconnected-(U1A-PF1-Pad31)
- U1 pad 32: GND -> controlSW23
- U1 pad 34: controlSW15 -> controlSW22
- U1 pad 35: controlSW16 -> controlSW21
- U1 pad 37: controlSW17 -> controlSW19
- U1 pad 4: Cline3 -> unconnected-(U1A-PD12-Pad4)
- U1 pad 5: Cline4 -> unconnected-(U1A-VDD-Pad5)
- U1 pad 7: VBAT -> unconnected-(U1A-BOOT0-Pad7)
- U1 pad 9: GND -> unconnected-(U1A-NC-Pad9)

Commit message: remove old power sheet
Connections:
- net VDD50USB renamed +5V
- U1 pad 16: VBAT -> +3V3
- U1 pad 33: VBAT -> +3V3
- U1 pad 47: VBAT -> VDDA
- U10 pad 4: VBAT -> VDDA
- U11 pad 4: VBAT -> VDDA
- U12 pad 4: VBAT -> VDDA
- U13 pad 4: VBAT -> VDDA
- U14 pad 4: VBAT -> VDDA
- U15 pad 4: VBAT -> VDDA
- U16 pad 4: VBAT -> VDDA
- U17 pad 4: VBAT -> VDDA
- U18 pad 4: VBAT -> VDDA
- U19 pad 4: VBAT -> VDDA
- U20 pad 4: VBAT -> VDDA
- U21 pad 4: VBAT -> VDDA
- U22 pad 4: VBAT -> VDDA
- U23 pad 4: VBAT -> VDDA
- U24 pad 4: VBAT -> VDDA
- U25 pad 4: VBAT -> VDDA
- U26 pad 4: VBAT -> VDDA
- U27 pad 4: VBAT -> VDDA
- U28 pad 4: VBAT -> VDDA
- U29 pad 4: VBAT -> VDDA
- U30 pad 4: VBAT -> VDDA
- U31 pad 4: VBAT -> VDDA
- U32 pad 4: VBAT -> VDDA
- U33 pad 4: VBAT -> VDDA
- U4 pad 16: VBAT -> +3V3
- U4 pad 6: VBAT -> +3V3
- U5 pad 16: VBAT -> +3V3
- U6 pad 16: VBAT -> +3V3
- U7 pad 15: VBAT -> VDDA
- U7 pad 16: VBAT -> +3V3
- U8 pad 15: VBAT -> VDDA
- U8 pad 16: VBAT -> +3V3
- U9 pad 15: VBAT -> VDDA
- U9 pad 16: VBAT -> +3V3

Commit message: initial column wiring
Parts:
- moved J3 473.5 mm to (145.7, 315.0)
- moved R32 327.9 mm to (135.0, 181.9), turned to -90 degrees
- moved Q20 327.0 mm to (135.2, 178.2), turned to 90 degrees
- moved D21 321.3 mm to (139.5, 178.2)
- moved K20 314.4 mm to (145.6, 181.7)
- moved Q19 260.6 mm to (142.3, 244.8), turned to 90 degrees
- moved D20 260.5 mm to (147.7, 243.6)
- moved R30 258.2 mm to (127.6, 245.4)
- moved K19 256.7 mm to (138.9, 250.0)
- moved R31 250.6 mm to (132.6, 259.9), turned to 90 degrees
- moved J2 223.6 mm to (369.1, 324.4)
- moved K18 113.6 mm to (249.0, 173.8)
- moved R28 105.3 mm to (238.8, 252.6)
- moved Q18 105.3 mm to (224.4, 204.9)
- moved R29 105.3 mm to (217.0, 204.9)
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Routing:
- net /Input Phone Jacks/ptTX16: track 0.00 -> 319.0 mm
- net /Input Phone Jacks/ptTX8: track 0.00 -> 277.4 mm
- net /Input Phone Jacks/ptTX0: track 0.00 -> 230.8 mm
- net /Input Phone Jacks/Line Control16/Tpbx: track 0.00 -> 95.7 mm
- net /Output Phone Jacks/Wiretap16/Tpots: track 0.00 -> 67.3 mm
- net /Input Phone Jacks/Tpbx0: track 0.00 -> 66.2 mm
- net /Output Phone Jacks/Wiretap8/Tpots: track 0.00 -> 60.7 mm
- net /Output Phone Jacks/Wiretap0/Tpots: track 0.00 -> 52.2 mm
- net /Input Phone Jacks/Line Control8/Tpbx: track 0.00 -> 51.1 mm
- net /Input Phone Jacks/Tpbx8: track 0.00 -> 49.9 mm
- net /Input Phone Jacks/Tpbx16: track 0.00 -> 41.1 mm
- net /Input Phone Jacks/Line Control0/Tpbx: track 0.00 -> 14.3 mm
- net Net-(D20-K): track 0.00 -> 11.8 mm
- net Net-(D4-K): track 0.00 -> 11.7 mm
- net Net-(D36-K): track 0.00 -> 11.1 mm
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