File: kicad/pbx-sniffer/pbx-sniffer.kicad_pcb (KiCad board)
At the start: 2 copper layers, 343 parts, among them K10 Relay_SPDT, K11 Relay_SPST-NO, K12 Relay_SPDT, K13 Relay_SPST-NO, K14 Relay_SPDT, K15 Relay_SPST-NO, K16 Relay_SPDT, K17 Relay_SPST-NO, K18 Relay_SPDT, K19 Relay_SPST-NO, K20 Relay_SPDT, K21 Relay_SPST-NO, K22 Relay_SPDT, K23 Relay_SPST-NO, K24 Relay_SPDT, K25 Relay_SPST-NO, K26 Relay_SPDT, K27 Relay_SPST-NO, K28 Relay_SPDT, K29 Relay_SPST-NO, K3 Relay_SPST-NO, K30 Relay_SPDT, K31 Relay_SPST-NO, K32 Relay_SPDT, K33 Relay_SPST-NO, K34 Relay_SPDT, K35 Relay_SPST-NO, K36 Relay_SPDT, K37 Relay_SPST-NO, K38 Relay_SPDT, K39 Relay_SPST-NO, K4 Relay_SPDT, K40 Relay_SPDT, K41 Relay_SPST-NO, K42 Relay_SPDT, K43 Relay_SPST-NO, K44 Relay_SPDT, K45 Relay_SPST-NO, K46 Relay_SPDT, K47 Relay_SPST-NO, K48 Relay_SPDT, K49 Relay_SPST-NO, K5 Relay_SPST-NO, K50 Relay_SPDT, K6 Relay_SPDT, K7 Relay_SPST-NO, K8 Relay_SPDT, K9 Relay_SPST-NO, Q10 PMOS, Q11 PMOS, Q12 PMOS, Q13 PMOS, Q14 PMOS, Q15 PMOS, Q16 PMOS, Q17 PMOS, Q18 PMOS, Q19 PMOS, Q20 PMOS, Q21 PMOS, Q22 PMOS, Q23 PMOS, Q24 PMOS, Q25 PMOS, Q26 PMOS, Q27 PMOS, Q28 PMOS, Q29 PMOS, Q3 PMOS, Q30 PMOS, Q31 PMOS, Q32 PMOS, Q33 PMOS, Q34 PMOS, Q35 PMOS, Q36 PMOS, Q37 PMOS, Q38 PMOS, Q39 PMOS, Q4 PMOS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

Commit message: organize jacks in the pcb layout
Parts:
- added J49: Conn_01x02_Socket, Connector_PinSocket_2.54mm:PinSocket_1x02_P2.54mm_Vertical, F.Cu at (518.3, 168.4)
- added J50: Conn_01x02_Socket, Connector_PinSocket_2.54mm:PinSocket_1x02_P2.54mm_Vertical, F.Cu at (522.9, 168.4)
- added J51: Conn_01x02_Socket, Connector_PinSocket_2.54mm:PinSocket_1x02_P2.54mm_Vertical, F.Cu at (527.5, 168.4)
- added J52: Conn_01x02_Socket, Connector_PinSocket_2.54mm:PinSocket_1x02_P2.54mm_Vertical, F.Cu at (532.1, 168.4)
- added J53: Conn_01x02_Socket, Connector_PinSocket_2.54mm:PinSocket_1x02_P2.54mm_Vertical, F.Cu at (518.3, 175.6)
- added J54: Conn_01x02_Socket, Connector_PinSocket_2.54mm:PinSocket_1x02_P2.54mm_Vertical, F.Cu at (522.9, 175.6)
- added J55: Conn_01x02_Socket, Connector_PinSocket_2.54mm:PinSocket_1x02_P2.54mm_Vertical, F.Cu at (527.5, 175.6)
- added J56: Conn_01x02_Socket, Connector_PinSocket_2.54mm:PinSocket_1x02_P2.54mm_Vertical, F.Cu at (532.1, 175.6)
- added J57: Conn_01x02_Socket, Connector_PinSocket_2.54mm:PinSocket_1x02_P2.54mm_Vertical, F.Cu at (518.3, 182.7)
- added J58: Conn_01x02_Socket, Connector_PinSocket_2.54mm:PinSocket_1x02_P2.54mm_Vertical, F.Cu at (522.9, 182.7)
- added J59: Conn_01x02_Socket, Connector_PinSocket_2.54mm:PinSocket_1x02_P2.54mm_Vertical, F.Cu at (527.5, 182.7)
- added J60: Conn_01x02_Socket, Connector_PinSocket_2.54mm:PinSocket_1x02_P2.54mm_Vertical, F.Cu at (532.1, 182.7)
- added J61: Conn_01x02_Socket, Connector_PinSocket_2.54mm:PinSocket_1x02_P2.54mm_Vertical, F.Cu at (518.3, 189.8)
- added J62: Conn_01x02_Socket, Connector_PinSocket_2.54mm:PinSocket_1x02_P2.54mm_Vertical, F.Cu at (522.9, 189.8)
- added J63: Conn_01x02_Socket, Connector_PinSocket_2.54mm:PinSocket_1x02_P2.54mm_Vertical, F.Cu at (527.5, 189.8)
- added J64: Conn_01x02_Socket, Connector_PinSocket_2.54mm:PinSocket_1x02_P2.54mm_Vertical, F.Cu at (532.1, 189.8)
- added R1: 10k, Resistor_THT:R_Axial_DIN0207_L6.3mm_D2.5mm_P10.16mm_Horizontal, F.Cu at (504.3, 168.1)
- added R102: 10k, Resistor_THT:R_Axial_DIN0207_L6.3mm_D2.5mm_P10.16mm_Horizontal, F.Cu at (504.3, 172.2)
- added R103: 10k, Resistor_THT:R_Axial_DIN0207_L6.3mm_D2.5mm_P10.16mm_Horizontal, F.Cu at (504.3, 176.2)
- added R104: 10k, Resistor_THT:R_Axial_DIN0207_L6.3mm_D2.5mm_P10.16mm_Horizontal, F.Cu at (504.3, 180.2)
- added R105: 10k, Resistor_THT:R_Axial_DIN0207_L6.3mm_D2.5mm_P10.16mm_Horizontal, F.Cu at (504.3, 184.3)
- added R106: 10k, Resistor_THT:R_Axial_DIN0207_L6.3mm_D2.5mm_P10.16mm_Horizontal, F.Cu at (504.3, 188.3)
- added R107: 10k, Resistor_THT:R_Axial_DIN0207_L6.3mm_D2.5mm_P10.16mm_Horizontal, F.Cu at (504.3, 192.4)
- added R108: 10k, Resistor_THT:R_Axial_DIN0207_L6.3mm_D2.5mm_P10.16mm_Horizontal, F.Cu at (504.3, 196.4)
- added R109: 10k, Resistor_THT:R_Axial_DIN0207_L6.3mm_D2.5mm_P10.16mm_Horizontal, F.Cu at (504.3, 200.5)
- added R110: 10k, Resistor_THT:R_Axial_DIN0207_L6.3mm_D2.5mm_P10.16mm_Horizontal, F.Cu at (504.3, 204.6)
- added R111: 10k, Resistor_THT:R_Axial_DIN0207_L6.3mm_D2.5mm_P10.16mm_Horizontal, F.Cu at (504.3, 208.6)
- added R112: 10k, Resistor_THT:R_Axial_DIN0207_L6.3mm_D2.5mm_P10.16mm_Horizontal, F.Cu at (504.3, 212.7)
- added R113: 10k, Resistor_THT:R_Axial_DIN0207_L6.3mm_D2.5mm_P10.16mm_Horizontal, F.Cu at (504.3, 216.7)
- added R114: 10k, Resistor_THT:R_Axial_DIN0207_L6.3mm_D2.5mm_P10.16mm_Horizontal, F.Cu at (504.3, 220.8)
- added R115: 10k, Resistor_THT:R_Axial_DIN0207_L6.3mm_D2.5mm_P10.16mm_Horizontal, F.Cu at (504.3, 224.8)
- added R116: 10k, Resistor_THT:R_Axial_DIN0207_L6.3mm_D2.5mm_P10.16mm_Horizontal, F.Cu at (504.3, 228.8)
- added U2: 74LS165, Package_DIP:DIP-16_W7.62mm, F.Cu at (517.6, 196.7)
- added U34: 74LS165, Package_DIP:DIP-16_W7.62mm, F.Cu at (528.4, 196.7)
- moved J1 508.1 mm to (143.1, 43.3), turned to 180 degrees
- moved J17 393.8 mm to (405.7, 43.3), turned to 180 degrees
- moved J41 390.4 mm to (388.1, 351.5), turned to 0 degrees
- moved J2 351.3 mm to (158.4, 43.3), turned to 180 degrees
- moved J4 298.6 mm to (192.3, 43.3), turned to 180 degrees
- moved J5 297.2 mm to (208.7, 43.3), turned to 180 degrees
- moved J6 295.8 mm to (225.2, 43.3), turned to 180 degrees
- moved J27 288.1 mm to (178.1, 351.5), turned to 0 degrees
- moved J31 277.4 mm to (238.1, 351.5), turned to 0 degrees
- moved J3 273.4 mm to (175.9, 43.3), turned to 180 degrees
- moved U1 268.0 mm to (276.0, 145.9)
- moved J7 264.2 mm to (241.6, 43.3), turned to 180 degrees
- moved J25 226.6 mm to (148.1, 351.5)
- moved J26 226.5 mm to (163.1, 351.5)
- moved J28 226.4 mm to (193.1, 351.5)
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Connections:
- net /multiplexer/LineControl0 renamed /Multiplexers/LineControl0
- net /multiplexer/LineControl1 renamed /Multiplexers/LineControl1
- net /multiplexer/LineControl10 renamed /Multiplexers/LineControl10
- net /multiplexer/LineControl11 renamed /Multiplexers/LineControl11
- net /multiplexer/LineControl12 renamed /Multiplexers/LineControl12
- net /multiplexer/LineControl13 renamed /Multiplexers/LineControl13
- net /multiplexer/LineControl14 renamed /Multiplexers/LineControl14
- net /multiplexer/LineControl15 renamed /Multiplexers/LineControl15
- net /multiplexer/LineControl16 renamed /Multiplexers/LineControl16
- net /multiplexer/LineControl17 renamed /Multiplexers/LineControl17
- net /multiplexer/LineControl18 renamed /Multiplexers/LineControl18
- net /multiplexer/LineControl19 renamed /Multiplexers/LineControl19
- net /multiplexer/LineControl2 renamed /Multiplexers/LineControl2
- net /multiplexer/LineControl20 renamed /Multiplexers/LineControl20
- net /multiplexer/LineControl21 renamed /Multiplexers/LineControl21
- net /multiplexer/LineControl22 renamed /Multiplexers/LineControl22
- net /multiplexer/LineControl23 renamed /Multiplexers/LineControl23
- net /multiplexer/LineControl3 renamed /Multiplexers/LineControl3
- net /multiplexer/LineControl4 renamed /Multiplexers/LineControl4
- net /multiplexer/LineControl5 renamed /Multiplexers/LineControl5
- net /multiplexer/LineControl6 renamed /Multiplexers/LineControl6
- net /multiplexer/LineControl7 renamed /Multiplexers/LineControl7
- net /multiplexer/LineControl8 renamed /Multiplexers/LineControl8
- net /multiplexer/LineControl9 renamed /Multiplexers/LineControl9
- net /multiplexer/Vss renamed /Multiplexers/Vss
- U1 pad 1: unconnected-(U1A-PC10-Pad1) -> shiftOut
- U1 pad 2: unconnected-(U1A-PC11-Pad2) -> shiftLd
- U1 pad 3: unconnected-(U1A-PC12-Pad3) -> shiftClk
- U1 pad 4: unconnected-(U1A-PD12-Pad4) -> shiftInh

Commit message: try organizing supporting components for first and second input jacks
Parts:
- moved U16 442.8 mm to (128.9, 99.5)
- moved R84 442.8 mm to (128.5, 95.4)
- moved R25 339.0 mm to (128.9, 85.0)
- moved K16 336.2 mm to (135.5, 65.3)
- moved D17 336.2 mm to (124.5, 81.2), turned to -90 degrees
- moved Q15 322.2 mm to (141.5, 100.5)
- moved K15 319.3 mm to (129.9, 90.5)
- moved R24 311.9 mm to (127.3, 110.0)
- moved JP8 311.3 mm to (124.0, 102.0), turned to -90 degrees
- moved D16 307.3 mm to (127.3, 106.5)
- moved R26 303.9 mm to (151.4, 119.0)
- moved Q16 303.0 mm to (169.0, 118.5)
- moved R28 183.8 mm to (162.1, 85.5), turned to 180 degrees
- moved D18 177.7 mm to (150.0, 88.7), turned to -90 degrees
- moved K17 175.8 mm to (154.5, 90.5)
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Routing:
- net /Input Phone Jacks/ptRX16: track 297.4 -> 105.7 mm, vias 2 -> 0
- net /Output Phone Jacks/Wiretap16/Tpots: track 67.3 -> 6.59 mm
- net /Input Phone Jacks/Rpbx16: track 297.4 -> 237.6 mm, vias 3 -> 1
- net /Input Phone Jacks/ptTX16: track 319.0 -> 269.8 mm
- net /Input Phone Jacks/ptTX8: track 277.4 -> 234.3 mm
- net /Input Phone Jacks/ptRX8: track 249.0 -> 209.2 mm, vias 2 -> 0
- net /Input Phone Jacks/Rpbx8: track 249.0 -> 212.2 mm, vias 3 -> 1
- net /Output Phone Jacks/Wiretap8/Tpots: track 60.7 -> 28.7 mm
- net /Input Phone Jacks/ptTX0: track 230.8 -> 219.4 mm
- net /Output Phone Jacks/Wiretap0/Tpots: track 52.2 -> 47.7 mm
- net /Input Phone Jacks/Rpbx0: track 18.2 -> 14.5 mm, vias 1 -> 0
- net /Input Phone Jacks/ptRX0: track 198.7 -> 195.0 mm, vias 2 -> 0

Commit message: initial module structure, for tiling later
Parts:
- moved D16 619.2 mm to (496.3, 603.9)
- moved D17 619.2 mm to (493.4, 578.5)
- moved D18 619.2 mm to (518.9, 586.0)
- moved D19 619.2 mm to (524.1, 603.8)
- moved JP8 619.2 mm to (492.9, 599.3)
- moved K16 619.2 mm to (504.4, 562.6)
- moved R26 619.2 mm to (520.3, 616.3)
- moved R27 619.2 mm to (524.8, 607.3)
- moved R84 619.2 mm to (497.4, 592.7)
- moved U16 619.2 mm to (497.8, 596.8)
- moved K15 619.2 mm to (498.8, 587.8)
- moved K17 619.2 mm to (523.4, 587.8)
- moved K18 619.2 mm to (527.4, 562.8)
- moved Q15 619.2 mm to (510.4, 597.8)
- moved Q16 619.2 mm to (537.9, 615.8)
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Connections:
- J1 pad 1: /Input Phone Jacks/ptTX6 -> /Input Phone Jacks/ptTX0
- J1 pad 2: /Input Phone Jacks/Line Control6/Tpbx -> /Input Phone Jacks/Line Control0/Tpbx
- J1 pad 3: /Input Phone Jacks/Rpbx6 -> /Input Phone Jacks/Rpbx0
- J1 pad 4: /Input Phone Jacks/ptRX6 -> /Input Phone Jacks/ptRX0
- J10 pad 1: /Input Phone Jacks/ptTX3 -> /Input Phone Jacks/ptTX9
- J10 pad 2: /Input Phone Jacks/Line Control3/Tpbx -> /Input Phone Jacks/Line Control9/Tpbx
- J10 pad 3: /Input Phone Jacks/Rpbx3 -> /Input Phone Jacks/Rpbx9
- J10 pad 4: /Input Phone Jacks/ptRX3 -> /Input Phone Jacks/ptRX9
- J11 pad 1: /Input Phone Jacks/ptTX4 -> /Input Phone Jacks/ptTX10
- J11 pad 2: /Input Phone Jacks/Line Control4/Tpbx -> /Input Phone Jacks/Line Control10/Tpbx
- J11 pad 3: /Input Phone Jacks/Rpbx4 -> /Input Phone Jacks/Rpbx10
- J11 pad 4: /Input Phone Jacks/ptRX4 -> /Input Phone Jacks/ptRX10
- J12 pad 1: /Input Phone Jacks/ptTX5 -> /Input Phone Jacks/ptTX11
- J12 pad 2: /Input Phone Jacks/Line Control5/Tpbx -> /Input Phone Jacks/Line Control11/Tpbx
- J12 pad 3: /Input Phone Jacks/Rpbx5 -> /Input Phone Jacks/Rpbx11
- J12 pad 4: /Input Phone Jacks/ptRX5 -> /Input Phone Jacks/ptRX11
- J2 pad 1: /Input Phone Jacks/ptTX7 -> /Input Phone Jacks/ptTX1
- J2 pad 2: /Input Phone Jacks/Line Control7/Tpbx -> /Input Phone Jacks/Line Control1/Tpbx
- J2 pad 3: /Input Phone Jacks/Rpbx7 -> /Input Phone Jacks/Rpbx1
- J2 pad 4: /Input Phone Jacks/ptRX7 -> /Input Phone Jacks/ptRX1
- J25 pad 1: /Input Phone Jacks/ptTX6 -> /Input Phone Jacks/ptTX0
- J25 pad 2: /Output Phone Jacks/Wiretap6/Tpots -> /Output Phone Jacks/Wiretap0/Tpots
- J25 pad 3: /Input Phone Jacks/Rpbx6 -> /Input Phone Jacks/Rpbx0
- J25 pad 4: /Input Phone Jacks/ptRX6 -> /Input Phone Jacks/ptRX0
- J26 pad 1: /Input Phone Jacks/ptTX7 -> /Input Phone Jacks/ptTX1
- J26 pad 2: /Output Phone Jacks/Wiretap7/Tpots -> /Output Phone Jacks/Wiretap1/Tpots
- J26 pad 3: /Input Phone Jacks/Rpbx7 -> /Input Phone Jacks/Rpbx1
- J26 pad 4: /Input Phone Jacks/ptRX7 -> /Input Phone Jacks/ptRX1
- J27 pad 1: /Input Phone Jacks/ptTX8 -> /Input Phone Jacks/ptTX2
- J27 pad 2: /Output Phone Jacks/Wiretap8/Tpots -> /Output Phone Jacks/Wiretap2/Tpots
- J27 pad 3: /Input Phone Jacks/Rpbx8 -> /Input Phone Jacks/Rpbx2
- J27 pad 4: /Input Phone Jacks/ptRX8 -> /Input Phone Jacks/ptRX2
- J28 pad 1: /Input Phone Jacks/ptTX9 -> /Input Phone Jacks/ptTX3
- J28 pad 2: /Output Phone Jacks/Wiretap9/Tpots -> /Output Phone Jacks/Wiretap3/Tpots
- J28 pad 3: /Input Phone Jacks/Rpbx9 -> /Input Phone Jacks/Rpbx3
- J28 pad 4: /Input Phone Jacks/ptRX9 -> /Input Phone Jacks/ptRX3
- J29 pad 1: /Input Phone Jacks/ptTX10 -> /Input Phone Jacks/ptTX4
- J29 pad 2: /Output Phone Jacks/Wiretap10/Tpots -> /Output Phone Jacks/Wiretap4/Tpots
- J29 pad 3: /Input Phone Jacks/Rpbx10 -> /Input Phone Jacks/Rpbx4
- J29 pad 4: /Input Phone Jacks/ptRX10 -> /Input Phone Jacks/ptRX4
- J3 pad 1: /Input Phone Jacks/ptTX8 -> /Input Phone Jacks/ptTX2
- J3 pad 2: /Input Phone Jacks/Line Control8/Tpbx -> /Input Phone Jacks/Line Control2/Tpbx
- J3 pad 3: /Input Phone Jacks/Rpbx8 -> /Input Phone Jacks/Rpbx2
- J3 pad 4: /Input Phone Jacks/ptRX8 -> /Input Phone Jacks/ptRX2
- J30 pad 1: /Input Phone Jacks/ptTX11 -> /Input Phone Jacks/ptTX5
- J30 pad 2: /Output Phone Jacks/Wiretap11/Tpots -> /Output Phone Jacks/Wiretap5/Tpots
- J30 pad 3: /Input Phone Jacks/Rpbx11 -> /Input Phone Jacks/Rpbx5
- J30 pad 4: /Input Phone Jacks/ptRX11 -> /Input Phone Jacks/ptRX5
- J31 pad 1: /Input Phone Jacks/ptTX0 -> /Input Phone Jacks/ptTX6
- J31 pad 2: /Output Phone Jacks/Wiretap0/Tpots -> /Output Phone Jacks/Wiretap6/Tpots
- J31 pad 3: /Input Phone Jacks/Rpbx0 -> /Input Phone Jacks/Rpbx6
- J31 pad 4: /Input Phone Jacks/ptRX0 -> /Input Phone Jacks/ptRX6
- J32 pad 1: /Input Phone Jacks/ptTX1 -> /Input Phone Jacks/ptTX7
- J32 pad 2: /Output Phone Jacks/Wiretap1/Tpots -> /Output Phone Jacks/Wiretap7/Tpots
- J32 pad 3: /Input Phone Jacks/Rpbx1 -> /Input Phone Jacks/Rpbx7
- J32 pad 4: /Input Phone Jacks/ptRX1 -> /Input Phone Jacks/ptRX7
- J33 pad 1: /Input Phone Jacks/ptTX2 -> /Input Phone Jacks/ptTX8
- J33 pad 2: /Output Phone Jacks/Wiretap2/Tpots -> /Output Phone Jacks/Wiretap8/Tpots
- J33 pad 3: /Input Phone Jacks/Rpbx2 -> /Input Phone Jacks/Rpbx8
- J33 pad 4: /Input Phone Jacks/ptRX2 -> /Input Phone Jacks/ptRX8
- J34 pad 1: /Input Phone Jacks/ptTX3 -> /Input Phone Jacks/ptTX9
- J34 pad 2: /Output Phone Jacks/Wiretap3/Tpots -> /Output Phone Jacks/Wiretap9/Tpots
- J34 pad 3: /Input Phone Jacks/Rpbx3 -> /Input Phone Jacks/Rpbx9
- J34 pad 4: /Input Phone Jacks/ptRX3 -> /Input Phone Jacks/ptRX9
- J35 pad 1: /Input Phone Jacks/ptTX4 -> /Input Phone Jacks/ptTX10
- J35 pad 2: /Output Phone Jacks/Wiretap4/Tpots -> /Output Phone Jacks/Wiretap10/Tpots
- J35 pad 3: /Input Phone Jacks/Rpbx4 -> /Input Phone Jacks/Rpbx10
- J35 pad 4: /Input Phone Jacks/ptRX4 -> /Input Phone Jacks/ptRX10
- J36 pad 1: /Input Phone Jacks/ptTX5 -> /Input Phone Jacks/ptTX11
- J36 pad 2: /Output Phone Jacks/Wiretap5/Tpots -> /Output Phone Jacks/Wiretap11/Tpots
- J36 pad 3: /Input Phone Jacks/Rpbx5 -> /Input Phone Jacks/Rpbx11
- J36 pad 4: /Input Phone Jacks/ptRX5 -> /Input Phone Jacks/ptRX11
- J4 pad 1: /Input Phone Jacks/ptTX9 -> /Input Phone Jacks/ptTX3
- J4 pad 2: /Input Phone Jacks/Line Control9/Tpbx -> /Input Phone Jacks/Line Control3/Tpbx
- J4 pad 3: /Input Phone Jacks/Rpbx9 -> /Input Phone Jacks/Rpbx3
- J4 pad 4: /Input Phone Jacks/ptRX9 -> /Input Phone Jacks/ptRX3
- J5 pad 1: /Input Phone Jacks/ptTX10 -> /Input Phone Jacks/ptTX4
- J5 pad 2: /Input Phone Jacks/Line Control10/Tpbx -> /Input Phone Jacks/Line Control4/Tpbx
- J5 pad 3: /Input Phone Jacks/Rpbx10 -> /Input Phone Jacks/Rpbx4
- J5 pad 4: /Input Phone Jacks/ptRX10 -> /Input Phone Jacks/ptRX4
- J6 pad 1: /Input Phone Jacks/ptTX11 -> /Input Phone Jacks/ptTX5
- J6 pad 2: /Input Phone Jacks/Line Control11/Tpbx -> /Input Phone Jacks/Line Control5/Tpbx
- J6 pad 3: /Input Phone Jacks/Rpbx11 -> /Input Phone Jacks/Rpbx5
- J6 pad 4: /Input Phone Jacks/ptRX11 -> /Input Phone Jacks/ptRX5
- J7 pad 1: /Input Phone Jacks/ptTX0 -> /Input Phone Jacks/ptTX6
- J7 pad 2: /Input Phone Jacks/Line Control0/Tpbx -> /Input Phone Jacks/Line Control6/Tpbx
- J7 pad 3: /Input Phone Jacks/Rpbx0 -> /Input Phone Jacks/Rpbx6
- J7 pad 4: /Input Phone Jacks/ptRX0 -> /Input Phone Jacks/ptRX6
- J8 pad 1: /Input Phone Jacks/ptTX1 -> /Input Phone Jacks/ptTX7
- J8 pad 2: /Input Phone Jacks/Line Control1/Tpbx -> /Input Phone Jacks/Line Control7/Tpbx
- J8 pad 3: /Input Phone Jacks/Rpbx1 -> /Input Phone Jacks/Rpbx7
- J8 pad 4: /Input Phone Jacks/ptRX1 -> /Input Phone Jacks/ptRX7
- J9 pad 1: /Input Phone Jacks/ptTX2 -> /Input Phone Jacks/ptTX8
- J9 pad 2: /Input Phone Jacks/Line Control2/Tpbx -> /Input Phone Jacks/Line Control8/Tpbx
- J9 pad 3: /Input Phone Jacks/Rpbx2 -> /Input Phone Jacks/Rpbx8
- J9 pad 4: /Input Phone Jacks/ptRX2 -> /Input Phone Jacks/ptRX8

Commit message: module modularized
Parts:
- moved U1 390.4 mm to (16.3, 211.3)
- moved R94 367.1 mm to (328.1, 404.8), turned to 0 degrees
- moved U26 363.4 mm to (328.5, 412.0), turned to 0 degrees
- moved JP18 362.5 mm to (333.1, 408.4), turned to 0 degrees
- moved R86 350.9 mm to (312.8, 404.8), turned to 0 degrees
- moved U18 347.3 mm to (313.2, 412.0), turned to 0 degrees
- moved JP10 346.5 mm to (317.8, 408.4), turned to 0 degrees
- moved Q36 336.1 mm to (331.4, 393.5), turned to 0 degrees
- moved R56 325.8 mm to (331.0, 381.8), turned to 0 degrees
- moved D37 325.3 mm to (312.9, 398.7)
- moved K36 306.6 mm to (321.0, 373.9)
- moved Q20 296.5 mm to (297.9, 393.5), turned to 0 degrees
- moved R54 289.0 mm to (331.0, 373.7)
- moved R32 285.9 mm to (297.5, 381.8), turned to 0 degrees
- moved D21 284.2 mm to (279.4, 398.7)
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Connections:
- K10 pad 3: unconnected-(K10-Pad3) -> Net-(JP30-B)
- K10 pad 4: /Input Phone Jacks/Line Control3/Tpbx -> Net-(JP30-A)
- K12 pad 3: unconnected-(K12-Pad3) -> Net-(JP31-B)
- K12 pad 4: /Input Phone Jacks/Line Control4/Tpbx -> Net-(JP31-A)
- K14 pad 3: unconnected-(K14-Pad3) -> Net-(JP32-B)
- K14 pad 4: /Input Phone Jacks/Line Control5/Tpbx -> Net-(JP32-A)
- K16 pad 3: unconnected-(K16-Pad3) -> Net-(JP33-B)
- K16 pad 4: /Input Phone Jacks/Line Control6/Tpbx -> Net-(JP33-A)
- K18 pad 3: unconnected-(K18-Pad3) -> Net-(JP34-B)
- K18 pad 4: /Input Phone Jacks/Line Control7/Tpbx -> Net-(JP34-A)
- K20 pad 3: unconnected-(K20-Pad3) -> Net-(JP35-B)
- K20 pad 4: /Input Phone Jacks/Line Control8/Tpbx -> Net-(JP35-A)
- K22 pad 3: unconnected-(K22-Pad3) -> Net-(JP36-B)
- K22 pad 4: /Input Phone Jacks/Line Control9/Tpbx -> Net-(JP36-A)
- K24 pad 3: unconnected-(K24-Pad3) -> Net-(JP37-B)
- K24 pad 4: /Input Phone Jacks/Line Control10/Tpbx -> Net-(JP37-A)
- K26 pad 3: unconnected-(K26-Pad3) -> Net-(JP38-B)
- K26 pad 4: /Input Phone Jacks/Line Control11/Tpbx -> Net-(JP38-A)
- K28 pad 3: unconnected-(K28-Pad3) -> Net-(JP39-B)
- K28 pad 4: /Input Phone Jacks/Line Control12/Tpbx -> Net-(JP39-A)
- K30 pad 3: unconnected-(K30-Pad3) -> Net-(JP40-B)
- K30 pad 4: /Input Phone Jacks/Line Control13/Tpbx -> Net-(JP40-A)
- K32 pad 3: unconnected-(K32-Pad3) -> Net-(JP41-B)
- K32 pad 4: /Input Phone Jacks/Line Control14/Tpbx -> Net-(JP41-A)
- K34 pad 3: unconnected-(K34-Pad3) -> Net-(JP42-B)
- K34 pad 4: /Input Phone Jacks/Line Control15/Tpbx -> Net-(JP42-A)
- K36 pad 3: unconnected-(K36-Pad3) -> Net-(JP43-B)
- K36 pad 4: /Input Phone Jacks/Line Control16/Tpbx -> Net-(JP43-A)
- K38 pad 3: unconnected-(K38-Pad3) -> Net-(JP44-B)
- K38 pad 4: /Input Phone Jacks/Line Control17/Tpbx -> Net-(JP44-A)
- K4 pad 3: unconnected-(K4-Pad3) -> Net-(JP27-B)
- K4 pad 4: /Input Phone Jacks/Line Control0/Tpbx -> Net-(JP27-A)
- K40 pad 3: unconnected-(K40-Pad3) -> Net-(JP45-B)
- K40 pad 4: /Input Phone Jacks/Line Control18/Tpbx -> Net-(JP45-A)
- K42 pad 3: unconnected-(K42-Pad3) -> Net-(JP46-B)
- K42 pad 4: /Input Phone Jacks/Line Control19/Tpbx -> Net-(JP46-A)
- K44 pad 3: unconnected-(K44-Pad3) -> Net-(JP47-B)
- K44 pad 4: /Input Phone Jacks/Line Control20/Tpbx -> Net-(JP47-A)
- K46 pad 3: unconnected-(K46-Pad3) -> Net-(JP48-B)
- K46 pad 4: /Input Phone Jacks/Line Control21/Tpbx -> Net-(JP48-A)
- K48 pad 3: unconnected-(K48-Pad3) -> Net-(JP49-B)
- K48 pad 4: /Input Phone Jacks/Line Control22/Tpbx -> Net-(JP49-A)
- K50 pad 3: unconnected-(K50-Pad3) -> Net-(JP50-B)
- K50 pad 4: /Input Phone Jacks/Line Control23/Tpbx -> Net-(JP50-A)
- K6 pad 3: unconnected-(K6-Pad3) -> Net-(JP28-B)
- K6 pad 4: /Input Phone Jacks/Line Control1/Tpbx -> Net-(JP28-A)
- K8 pad 3: unconnected-(K8-Pad3) -> Net-(JP29-B)
- K8 pad 4: /Input Phone Jacks/Line Control2/Tpbx -> Net-(JP29-A)
- Q10 pad 2: controlSW3 -> /Multiplexers/LineControl3
- Q11 pad 2: /hookSW4 -> hookSW4
- Q12 pad 2: controlSW4 -> /Multiplexers/LineControl4
- Q13 pad 2: /hookSW5 -> hookSW5
- Q14 pad 2: controlSW5 -> /Multiplexers/LineControl5
- Q15 pad 2: /hookSW6 -> hookSW6
- Q16 pad 2: controlSW6 -> /Multiplexers/LineControl6
- Q17 pad 2: /hookSW7 -> hookSW7
- Q18 pad 2: controlSW7 -> /Multiplexers/LineControl7
- Q19 pad 2: /hookSW8 -> hookSW8
- Q20 pad 2: controlSW8 -> /Multiplexers/LineControl8
- Q21 pad 2: /hookSW9 -> hookSW9
- Q22 pad 2: controlSW9 -> /Multiplexers/LineControl9
- Q23 pad 2: /hookSW10 -> hookSW10
- Q24 pad 2: controlSW10 -> /Multiplexers/LineControl10
- Q25 pad 2: /hookSW11 -> hookSW11
- Q26 pad 2: controlSW11 -> /Multiplexers/LineControl11
- Q27 pad 2: /hookSW12 -> hookSW12
- Q28 pad 2: controlSW12 -> /Multiplexers/LineControl12
- Q29 pad 2: /hookSW13 -> hookSW13
- Q3 pad 2: /hookSW0 -> hookSW0
- Q30 pad 2: controlSW13 -> /Multiplexers/LineControl13
- Q31 pad 2: /hookSW14 -> hookSW14
- Q32 pad 2: controlSW14 -> /Multiplexers/LineControl14
- Q33 pad 2: /hookSW15 -> hookSW15
- Q34 pad 2: controlSW15 -> /Multiplexers/LineControl15
- Q35 pad 2: /hookSW16 -> hookSW16
- Q36 pad 2: controlSW16 -> /Multiplexers/LineControl16
- Q37 pad 2: /hookSW17 -> hookSW17
- Q38 pad 2: controlSW17 -> /Multiplexers/LineControl17
- Q39 pad 2: /hookSW18 -> hookSW18
- Q4 pad 2: controlSW0 -> /Multiplexers/LineControl0
- Q40 pad 2: controlSW18 -> /Multiplexers/LineControl18
- Q41 pad 2: /hookSW19 -> hookSW19
- Q42 pad 2: controlSW19 -> /Multiplexers/LineControl19
- Q43 pad 2: /hookSW20 -> hookSW20
- Q44 pad 2: controlSW20 -> /Multiplexers/LineControl20
- Q45 pad 2: /hookSW21 -> hookSW21
- Q46 pad 2: controlSW21 -> /Multiplexers/LineControl21
- Q47 pad 2: /hookSW22 -> hookSW22
- Q48 pad 2: controlSW22 -> /Multiplexers/LineControl22
- Q49 pad 2: /hookSW23 -> hookSW23
- Q5 pad 2: /hookSW1 -> hookSW1
- Q50 pad 2: controlSW23 -> /Multiplexers/LineControl23
- Q6 pad 2: controlSW1 -> /Multiplexers/LineControl1
- Q7 pad 2: /hookSW2 -> hookSW2
- Q8 pad 2: controlSW2 -> /Multiplexers/LineControl2
- Q9 pad 2: /hookSW3 -> hookSW3
- R11 pad 1: controlSW1 -> /Multiplexers/LineControl1
- R12 pad 2: /hookSW2 -> hookSW2
- R14 pad 1: controlSW2 -> /Multiplexers/LineControl2
- R15 pad 2: /hookSW3 -> hookSW3
- R17 pad 1: controlSW3 -> /Multiplexers/LineControl3
- R18 pad 2: /hookSW4 -> hookSW4
- R20 pad 1: controlSW4 -> /Multiplexers/LineControl4
- R21 pad 2: /hookSW5 -> hookSW5
- R23 pad 1: controlSW5 -> /Multiplexers/LineControl5
- R24 pad 2: /hookSW6 -> hookSW6
- R26 pad 1: controlSW6 -> /Multiplexers/LineControl6
- R27 pad 2: /hookSW7 -> hookSW7
- R29 pad 1: controlSW7 -> /Multiplexers/LineControl7
- R30 pad 2: /hookSW8 -> hookSW8
- R32 pad 1: controlSW8 -> /Multiplexers/LineControl8
- R33 pad 2: /hookSW9 -> hookSW9
- R35 pad 1: controlSW9 -> /Multiplexers/LineControl9
- R36 pad 2: /hookSW10 -> hookSW10
- R38 pad 1: controlSW10 -> /Multiplexers/LineControl10
- R39 pad 2: /hookSW11 -> hookSW11
- R41 pad 1: controlSW11 -> /Multiplexers/LineControl11
- R42 pad 2: /hookSW12 -> hookSW12
- R44 pad 1: controlSW12 -> /Multiplexers/LineControl12
- R45 pad 2: /hookSW13 -> hookSW13
- R47 pad 1: controlSW13 -> /Multiplexers/LineControl13
- R48 pad 2: /hookSW14 -> hookSW14
- R50 pad 1: controlSW14 -> /Multiplexers/LineControl14
- R51 pad 2: /hookSW15 -> hookSW15
- R53 pad 1: controlSW15 -> /Multiplexers/LineControl15
- R54 pad 2: /hookSW16 -> hookSW16
- R56 pad 1: controlSW16 -> /Multiplexers/LineControl16
- R57 pad 2: /hookSW17 -> hookSW17
- R59 pad 1: controlSW17 -> /Multiplexers/LineControl17
- R6 pad 2: /hookSW0 -> hookSW0
- R60 pad 2: /hookSW18 -> hookSW18
- R62 pad 1: controlSW18 -> /Multiplexers/LineControl18
- R63 pad 2: /hookSW19 -> hookSW19
- R65 pad 1: controlSW19 -> /Multiplexers/LineControl19
- R66 pad 2: /hookSW20 -> hookSW20
- R68 pad 1: controlSW20 -> /Multiplexers/LineControl20
- R69 pad 2: /hookSW21 -> hookSW21
- R71 pad 1: controlSW21 -> /Multiplexers/LineControl21
- R72 pad 2: /hookSW22 -> hookSW22
- R74 pad 1: controlSW22 -> /Multiplexers/LineControl22
- R75 pad 2: /hookSW23 -> hookSW23
- R77 pad 1: controlSW23 -> /Multiplexers/LineControl23
- R8 pad 1: controlSW0 -> /Multiplexers/LineControl0
- R9 pad 2: /hookSW1 -> hookSW1
- U1 pad 19: GND -> GNDD
- U1 pad 20: GND -> GNDD
- U1 pad 22: GND -> GNDD
- U1 pad 32: controlSW23 -> hookSW23
- U1 pad 34: controlSW22 -> hookSW22
- U1 pad 35: controlSW21 -> hookSW21
- U1 pad 36: controlSW20 -> hookSW20
- U1 pad 37: controlSW19 -> hookSW19
- U1 pad 38: controlSW18 -> hookSW18
- U1 pad 49: GND -> GNDD
- U1 pad 57: controlSW0 -> hookSW0
- U1 pad 58: controlSW1 -> hookSW1
- U1 pad 59: controlSW2 -> hookSW2
- U1 pad 60: GND -> GNDD
- U1 pad 61: controlSW3 -> hookSW3
- U1 pad 62: controlSW4 -> hookSW4
- U1 pad 63: controlSW5 -> hookSW5
- U1 pad 64: controlSW6 -> hookSW6
- U1 pad 65: controlSW7 -> hookSW7
- U1 pad 66: controlSW8 -> hookSW8
- U1 pad 67: controlSW9 -> hookSW9
- U1 pad 68: controlSW10 -> hookSW10
- U1 pad 69: controlSW11 -> hookSW11
- U1 pad 70: controlSW12 -> hookSW12
- U1 pad 71: controlSW13 -> hookSW13
- U1 pad 72: GND -> GNDD
- U1 pad 73: controlSW14 -> hookSW14
- U1 pad 74: controlSW15 -> hookSW15
- U1 pad 75: controlSW16 -> hookSW16
- U1 pad 77: controlSW17 -> hookSW17
- U1 pad 8: GND -> GNDD
- U4 pad 8: /Multiplexers/Vss -> GNDD
- U5 pad 4: /Multiplexers/Vss -> GNDD
- U5 pad 8: /Multiplexers/Vss -> GNDD
- U6 pad 5: /Multiplexers/Vss -> GNDD
- U6 pad 8: /Multiplexers/Vss -> GNDD
- U7 pad 14: /ADC/AGND -> GNDD
- U7 pad 9: /ADC/DGND -> GNDD
- U8 pad 14: /ADC/AGND -> GNDD
- U8 pad 9: /ADC/DGND -> GNDD
- U9 pad 14: /ADC/AGND -> GNDD
- U9 pad 9: /ADC/DGND -> GNDD
Routing:
- net /Input Phone Jacks/ptTX16: track 269.8 -> 0.00 mm
- net /Input Phone Jacks/Rpbx16: track 237.6 -> 0.00 mm, vias 1 -> 0
- net /Input Phone Jacks/ptTX8: track 234.3 -> 0.00 mm
- net /Input Phone Jacks/Rpbx8: track 212.2 -> 0.00 mm, vias 1 -> 0
- net /Input Phone Jacks/ptRX8: track 209.2 -> 0.00 mm
- net /Input Phone Jacks/Line Control16/Tpbx: track 173.6 -> 0.00 mm
- net /Input Phone Jacks/ptTX0: track 219.4 -> 91.4 mm, vias 0 -> 5
- net /Input Phone Jacks/Line Control8/Tpbx: track 123.0 -> 0.00 mm
- net /Input Phone Jacks/ptRX16: track 105.7 -> 0.00 mm
- net /Input Phone Jacks/ptRX0: track 195.0 -> 92.3 mm, vias 0 -> 4
- net /Input Phone Jacks/Rpbx0: track 14.5 -> 77.4 mm, vias 0 -> 3
- net /ADC/ADC0: track 0.00 -> 57.9 mm
- net /ADC/ADC23: track 0.00 -> 57.2 mm
- net /Input Phone Jacks/Tpbx0: track 66.2 -> 13.2 mm
- net /ADC/ADC22: track 0.00 -> 51.6 mm
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- added copper zone on B.Cu, net GNDA
- added copper zone on F.Cu, net GNDA
- added copper zone on B.Cu, net GNDD
- added copper zone on B.Cu, net VDDA
