File: kicad/pbx-sniffer/pbx-sniffer.kicad_pcb (KiCad board)
At the start: 2 copper layers, 401 parts, among them J49 Conn_01x02_Socket, J50 Conn_01x02_Socket, J51 Conn_01x02_Socket, J52 Conn_01x02_Socket, J53 Conn_01x02_Socket, J54 Conn_01x02_Socket, J55 Conn_01x02_Socket, J56 Conn_01x02_Socket, J57 Conn_01x02_Socket, J58 Conn_01x02_Socket, J59 Conn_01x02_Socket, J60 Conn_01x02_Socket, J61 Conn_01x02_Socket, J62 Conn_01x02_Socket, J63 Conn_01x02_Socket, J64 Conn_01x02_Socket, K10 Relay_SPDT, K11 Relay_SPST-NO, K12 Relay_SPDT, K13 Relay_SPST-NO, K14 Relay_SPDT, K15 Relay_SPST-NO, K16 Relay_SPDT, K17 Relay_SPST-NO, K18 Relay_SPDT, K19 Relay_SPST-NO, K20 Relay_SPDT, K21 Relay_SPST-NO, K22 Relay_SPDT, K23 Relay_SPST-NO, K24 Relay_SPDT, K25 Relay_SPST-NO, K26 Relay_SPDT, K27 Relay_SPST-NO, K28 Relay_SPDT, K29 Relay_SPST-NO, K3 Relay_SPST-NO, K30 Relay_SPDT, K31 Relay_SPST-NO, K32 Relay_SPDT, K33 Relay_SPST-NO, K34 Relay_SPDT, K35 Relay_SPST-NO, K36 Relay_SPDT, K37 Relay_SPST-NO, K38 Relay_SPDT, K39 Relay_SPST-NO, K4 Relay_SPDT, K40 Relay_SPDT, K41 Relay_SPST-NO, K42 Relay_SPDT, K43 Relay_SPST-NO, K44 Relay_SPDT, K45 Relay_SPST-NO, K46 Relay_SPDT, K47 Relay_SPST-NO, K48 Relay_SPDT, K49 Relay_SPST-NO, K5 Relay_SPST-NO, K50 Relay_SPDT, K6 Relay_SPDT, K7 Relay_SPST-NO, K8 Relay_SPDT, K9 Relay_SPST-NO, Q10 PMOS, Q11 PMOS, Q12 PMOS, Q13 PMOS, Q14 PMOS, Q15 PMOS, Q16 PMOS, Q17 PMOS, Q18 PMOS, Q19 PMOS, Q20 PMOS, Q21 PMOS, Q22 PMOS, Q23 PMOS, Q24 PMOS, Q25 PMOS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

Commit message: quickly try laying out pcb with plugins
Parts:
- JP28, JP29, JP30, JP31, JP32, JP33, JP34, JP35, JP36, JP37, JP38, JP39, JP40, JP41, JP42, JP43, JP44, JP45, JP46, JP47, JP48, JP49, JP50: moved to B.Cu
- moved R84 563.3 mm to (182.1, 125.9), turned to 90 degrees
- moved R81 530.4 mm to (131.1, 125.9), turned to 90 degrees
- moved Q16 508.5 mm to (239.1, 204.3), turned to 180 degrees
- moved D19 503.3 mm to (253.9, 179.2)
- moved Q18 497.3 mm to (256.1, 204.3), turned to 180 degrees
- moved K50 494.4 mm to (532.4, 182.6)
- moved JP8 492.6 mm to (249.3, 171.2)
- moved U16 492.5 mm to (246.8, 173.1), turned to 180 degrees
- moved D51 491.7 mm to (525.9, 179.2)
- moved R79 478.9 mm to (97.1, 125.9), turned to 90 degrees
- moved K49 477.3 mm to (532.6, 218.9), turned to 90 degrees
- moved JP4 474.9 mm to (181.3, 171.2), turned to -90 degrees
- moved D17 474.6 mm to (236.9, 179.2), turned to 0 degrees
- moved R76 474.4 mm to (535.5, 225.0), turned to 180 degrees
- moved Q50 474.3 mm to (528.1, 204.3), turned to 180 degrees
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Connections:
- K10 pad 3: Net-(JP30-B) -> unconnected-(K10-Pad3)
- K10 pad 4: Net-(JP30-A) -> /Input Phone Jacks/Line Control3/Tpbx
- K12 pad 3: Net-(JP31-B) -> unconnected-(K12-Pad3)
- K12 pad 4: Net-(JP31-A) -> /Input Phone Jacks/Line Control4/Tpbx
- K14 pad 3: Net-(JP32-B) -> unconnected-(K14-Pad3)
- K14 pad 4: Net-(JP32-A) -> /Input Phone Jacks/Line Control5/Tpbx
- K16 pad 3: Net-(JP33-B) -> unconnected-(K16-Pad3)
- K16 pad 4: Net-(JP33-A) -> /Input Phone Jacks/Line Control6/Tpbx
- K18 pad 3: Net-(JP34-B) -> unconnected-(K18-Pad3)
- K18 pad 4: Net-(JP34-A) -> /Input Phone Jacks/Line Control7/Tpbx
- K20 pad 3: Net-(JP35-B) -> unconnected-(K20-Pad3)
- K20 pad 4: Net-(JP35-A) -> /Input Phone Jacks/Line Control8/Tpbx
- K22 pad 3: Net-(JP36-B) -> unconnected-(K22-Pad3)
- K22 pad 4: Net-(JP36-A) -> /Input Phone Jacks/Line Control9/Tpbx
- K24 pad 3: Net-(JP37-B) -> unconnected-(K24-Pad3)
- K24 pad 4: Net-(JP37-A) -> /Input Phone Jacks/Line Control10/Tpbx
- K26 pad 3: Net-(JP38-B) -> unconnected-(K26-Pad3)
- K26 pad 4: Net-(JP38-A) -> /Input Phone Jacks/Line Control11/Tpbx
- K28 pad 3: Net-(JP39-B) -> unconnected-(K28-Pad3)
- K28 pad 4: Net-(JP39-A) -> /Input Phone Jacks/Line Control12/Tpbx
- K30 pad 3: Net-(JP40-B) -> unconnected-(K30-Pad3)
- K30 pad 4: Net-(JP40-A) -> /Input Phone Jacks/Line Control13/Tpbx
- K32 pad 3: Net-(JP41-B) -> unconnected-(K32-Pad3)
- K32 pad 4: Net-(JP41-A) -> /Input Phone Jacks/Line Control14/Tpbx
- K34 pad 3: Net-(JP42-B) -> unconnected-(K34-Pad3)
- K34 pad 4: Net-(JP42-A) -> /Input Phone Jacks/Line Control15/Tpbx
- K36 pad 3: Net-(JP43-B) -> unconnected-(K36-Pad3)
- K36 pad 4: Net-(JP43-A) -> /Input Phone Jacks/Line Control16/Tpbx
- K38 pad 3: Net-(JP44-B) -> unconnected-(K38-Pad3)
- K38 pad 4: Net-(JP44-A) -> /Input Phone Jacks/Line Control17/Tpbx
- K4 pad 3: Net-(JP27-B) -> unconnected-(K4-Pad3)
- K4 pad 4: Net-(JP27-A) -> /Input Phone Jacks/Line Control0/Tpbx
- K40 pad 3: Net-(JP45-B) -> unconnected-(K40-Pad3)
- K40 pad 4: Net-(JP45-A) -> /Input Phone Jacks/Line Control18/Tpbx
- K42 pad 3: Net-(JP46-B) -> unconnected-(K42-Pad3)
- K42 pad 4: Net-(JP46-A) -> /Input Phone Jacks/Line Control19/Tpbx
- K44 pad 3: Net-(JP47-B) -> unconnected-(K44-Pad3)
- K44 pad 4: Net-(JP47-A) -> /Input Phone Jacks/Line Control20/Tpbx
- K46 pad 3: Net-(JP48-B) -> unconnected-(K46-Pad3)
- K46 pad 4: Net-(JP48-A) -> /Input Phone Jacks/Line Control21/Tpbx
- K48 pad 3: Net-(JP49-B) -> unconnected-(K48-Pad3)
- K48 pad 4: Net-(JP49-A) -> /Input Phone Jacks/Line Control22/Tpbx
- K50 pad 3: Net-(JP50-B) -> unconnected-(K50-Pad3)
- K50 pad 4: Net-(JP50-A) -> /Input Phone Jacks/Line Control23/Tpbx
- K6 pad 3: Net-(JP28-B) -> unconnected-(K6-Pad3)
- K6 pad 4: Net-(JP28-A) -> /Input Phone Jacks/Line Control1/Tpbx
- K8 pad 3: Net-(JP29-B) -> unconnected-(K8-Pad3)
- K8 pad 4: Net-(JP29-A) -> /Input Phone Jacks/Line Control2/Tpbx
- Q10 pad 2: /Multiplexers/LineControl3 -> controlSW3
- Q11 pad 2: hookSW4 -> /hookSW4
- Q12 pad 2: /Multiplexers/LineControl4 -> controlSW4
- Q13 pad 2: hookSW5 -> /hookSW5
- Q14 pad 2: /Multiplexers/LineControl5 -> controlSW5
- Q15 pad 2: hookSW6 -> /hookSW6
- Q16 pad 2: /Multiplexers/LineControl6 -> controlSW6
- Q17 pad 2: hookSW7 -> /hookSW7
- Q18 pad 2: /Multiplexers/LineControl7 -> controlSW7
- Q19 pad 2: hookSW8 -> /hookSW8
- Q20 pad 2: /Multiplexers/LineControl8 -> controlSW8
- Q21 pad 2: hookSW9 -> /hookSW9
- Q22 pad 2: /Multiplexers/LineControl9 -> controlSW9
- Q23 pad 2: hookSW10 -> /hookSW10
- Q24 pad 2: /Multiplexers/LineControl10 -> controlSW10
- Q25 pad 2: hookSW11 -> /hookSW11
- Q26 pad 2: /Multiplexers/LineControl11 -> controlSW11
- Q27 pad 2: hookSW12 -> /hookSW12
- Q28 pad 2: /Multiplexers/LineControl12 -> controlSW12
- Q29 pad 2: hookSW13 -> /hookSW13
- Q3 pad 2: hookSW0 -> /hookSW0
- Q30 pad 2: /Multiplexers/LineControl13 -> controlSW13
- Q31 pad 2: hookSW14 -> /hookSW14
- Q32 pad 2: /Multiplexers/LineControl14 -> controlSW14
- Q33 pad 2: hookSW15 -> /hookSW15
- Q34 pad 2: /Multiplexers/LineControl15 -> controlSW15
- Q35 pad 2: hookSW16 -> /hookSW16
- Q36 pad 2: /Multiplexers/LineControl16 -> controlSW16
- Q37 pad 2: hookSW17 -> /hookSW17
- Q38 pad 2: /Multiplexers/LineControl17 -> controlSW17
- Q39 pad 2: hookSW18 -> /hookSW18
- Q4 pad 2: /Multiplexers/LineControl0 -> controlSW0
- Q40 pad 2: /Multiplexers/LineControl18 -> controlSW18
- Q41 pad 2: hookSW19 -> /hookSW19
- Q42 pad 2: /Multiplexers/LineControl19 -> controlSW19
- Q43 pad 2: hookSW20 -> /hookSW20
- Q44 pad 2: /Multiplexers/LineControl20 -> controlSW20
- Q45 pad 2: hookSW21 -> /hookSW21
- Q46 pad 2: /Multiplexers/LineControl21 -> controlSW21
- Q47 pad 2: hookSW22 -> /hookSW22
- Q48 pad 2: /Multiplexers/LineControl22 -> controlSW22
- Q49 pad 2: hookSW23 -> /hookSW23
- Q5 pad 2: hookSW1 -> /hookSW1
- Q50 pad 2: /Multiplexers/LineControl23 -> controlSW23
- Q6 pad 2: /Multiplexers/LineControl1 -> controlSW1
- Q7 pad 2: hookSW2 -> /hookSW2
- Q8 pad 2: /Multiplexers/LineControl2 -> controlSW2
- Q9 pad 2: hookSW3 -> /hookSW3
- R11 pad 1: /Multiplexers/LineControl1 -> controlSW1
- R12 pad 2: hookSW2 -> /hookSW2
- R14 pad 1: /Multiplexers/LineControl2 -> controlSW2
- R15 pad 2: hookSW3 -> /hookSW3
- R17 pad 1: /Multiplexers/LineControl3 -> controlSW3
- R18 pad 2: hookSW4 -> /hookSW4
- R20 pad 1: /Multiplexers/LineControl4 -> controlSW4
- R21 pad 2: hookSW5 -> /hookSW5
- R23 pad 1: /Multiplexers/LineControl5 -> controlSW5
- R24 pad 2: hookSW6 -> /hookSW6
- R26 pad 1: /Multiplexers/LineControl6 -> controlSW6
- R27 pad 2: hookSW7 -> /hookSW7
- R29 pad 1: /Multiplexers/LineControl7 -> controlSW7
- R30 pad 2: hookSW8 -> /hookSW8
- R32 pad 1: /Multiplexers/LineControl8 -> controlSW8
- R33 pad 2: hookSW9 -> /hookSW9
- R35 pad 1: /Multiplexers/LineControl9 -> controlSW9
- R36 pad 2: hookSW10 -> /hookSW10
- R38 pad 1: /Multiplexers/LineControl10 -> controlSW10
- R39 pad 2: hookSW11 -> /hookSW11
- R41 pad 1: /Multiplexers/LineControl11 -> controlSW11
- R42 pad 2: hookSW12 -> /hookSW12
- R44 pad 1: /Multiplexers/LineControl12 -> controlSW12
- R45 pad 2: hookSW13 -> /hookSW13
- R47 pad 1: /Multiplexers/LineControl13 -> controlSW13
- R48 pad 2: hookSW14 -> /hookSW14
- R50 pad 1: /Multiplexers/LineControl14 -> controlSW14
- R51 pad 2: hookSW15 -> /hookSW15
- R53 pad 1: /Multiplexers/LineControl15 -> controlSW15
- R54 pad 2: hookSW16 -> /hookSW16
- R56 pad 1: /Multiplexers/LineControl16 -> controlSW16
- R57 pad 2: hookSW17 -> /hookSW17
- R59 pad 1: /Multiplexers/LineControl17 -> controlSW17
- R6 pad 2: hookSW0 -> /hookSW0
- R60 pad 2: hookSW18 -> /hookSW18
- R62 pad 1: /Multiplexers/LineControl18 -> controlSW18
- R63 pad 2: hookSW19 -> /hookSW19
- R65 pad 1: /Multiplexers/LineControl19 -> controlSW19
- R66 pad 2: hookSW20 -> /hookSW20
- R68 pad 1: /Multiplexers/LineControl20 -> controlSW20
- R69 pad 2: hookSW21 -> /hookSW21
- R71 pad 1: /Multiplexers/LineControl21 -> controlSW21
- R72 pad 2: hookSW22 -> /hookSW22
- R74 pad 1: /Multiplexers/LineControl22 -> controlSW22
- R75 pad 2: hookSW23 -> /hookSW23
- R77 pad 1: /Multiplexers/LineControl23 -> controlSW23
- R8 pad 1: /Multiplexers/LineControl0 -> controlSW0
- R9 pad 2: hookSW1 -> /hookSW1
- U1 pad 19: GNDD -> GND
- U1 pad 20: GNDD -> GND
- U1 pad 22: GNDD -> GND
- U1 pad 32: hookSW23 -> controlSW23
- U1 pad 34: hookSW22 -> controlSW22
- U1 pad 35: hookSW21 -> controlSW21
- U1 pad 36: hookSW20 -> controlSW20
- U1 pad 37: hookSW19 -> controlSW19
- U1 pad 38: hookSW18 -> controlSW18
- U1 pad 49: GNDD -> GND
- U1 pad 57: hookSW0 -> controlSW0
- U1 pad 58: hookSW1 -> controlSW1
- U1 pad 59: hookSW2 -> controlSW2
- U1 pad 60: GNDD -> GND
- U1 pad 61: hookSW3 -> controlSW3
- U1 pad 62: hookSW4 -> controlSW4
- U1 pad 63: hookSW5 -> controlSW5
- U1 pad 64: hookSW6 -> controlSW6
- U1 pad 65: hookSW7 -> controlSW7
- U1 pad 66: hookSW8 -> controlSW8
- U1 pad 67: hookSW9 -> controlSW9
- U1 pad 68: hookSW10 -> controlSW10
- U1 pad 69: hookSW11 -> controlSW11
- U1 pad 70: hookSW12 -> controlSW12
- U1 pad 71: hookSW13 -> controlSW13
- U1 pad 72: GNDD -> GND
- U1 pad 73: hookSW14 -> controlSW14
- U1 pad 74: hookSW15 -> controlSW15
- U1 pad 75: hookSW16 -> controlSW16
- U1 pad 77: hookSW17 -> controlSW17
- U1 pad 8: GNDD -> GND
- U4 pad 8: GNDD -> /Multiplexers/Vss
- U5 pad 4: GNDD -> /Multiplexers/Vss
- U5 pad 8: GNDD -> /Multiplexers/Vss
- U6 pad 5: GNDD -> /Multiplexers/Vss
- U6 pad 8: GNDD -> /Multiplexers/Vss
- U7 pad 14: GNDD -> /ADC/AGND
- U7 pad 9: GNDD -> /ADC/DGND
- U8 pad 14: GNDD -> /ADC/AGND
- U8 pad 9: GNDD -> /ADC/DGND
- U9 pad 14: GNDD -> /ADC/AGND
- U9 pad 9: GNDD -> /ADC/DGND
Routing:
- net /Input Phone Jacks/ptRX0: track 92.3 -> 2031.0 mm, vias 4 -> 88
- net /Input Phone Jacks/ptRX1: track 0.00 -> 92.3 mm, vias 0 -> 4
- net /Input Phone Jacks/ptRX2: track 0.00 -> 92.3 mm, vias 0 -> 4
- net /Input Phone Jacks/ptTX20: track 0.00 -> 91.4 mm, vias 0 -> 5
- net /Input Phone Jacks/ptTX17: track 0.00 -> 91.4 mm, vias 0 -> 5
- net /Input Phone Jacks/ptTX14: track 0.00 -> 91.4 mm, vias 0 -> 5
- net /Input Phone Jacks/ptTX11: track 0.00 -> 91.4 mm, vias 0 -> 5
- net /Input Phone Jacks/ptTX9: track 0.00 -> 91.4 mm, vias 0 -> 5
- net /Input Phone Jacks/ptTX7: track 0.00 -> 91.4 mm, vias 0 -> 5
- net /Input Phone Jacks/ptTX21: track 0.00 -> 91.4 mm, vias 0 -> 5
- net /Input Phone Jacks/ptTX19: track 0.00 -> 91.4 mm, vias 0 -> 5
- net /Input Phone Jacks/ptTX18: track 0.00 -> 91.4 mm, vias 0 -> 5
- net /Input Phone Jacks/ptTX16: track 0.00 -> 91.4 mm, vias 0 -> 5
- net /Input Phone Jacks/ptTX15: track 0.00 -> 91.4 mm, vias 0 -> 5
- net /Input Phone Jacks/ptTX13: track 0.00 -> 91.4 mm, vias 0 -> 5
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
Commit message: copy pasted traces
Routing:
- net /Input Phone Jacks/ptRX0: track 2031.0 -> 92.3 mm, vias 88 -> 4
- net /ADC/ADC3: track 74.5 -> 219.2 mm
- net unconnected-(K4-Pad3): track 12.4 -> 148.8 mm
- net /Input Phone Jacks/ptRX23: track 0.00 -> 92.3 mm, vias 0 -> 4
- net /Input Phone Jacks/ptRX22: track 0.00 -> 92.3 mm, vias 0 -> 4
- net /Input Phone Jacks/ptRX4: track 0.00 -> 92.3 mm, vias 0 -> 4
- net /Input Phone Jacks/ptRX5: track 0.00 -> 92.3 mm, vias 0 -> 4
- net /Input Phone Jacks/ptRX3: track 0.00 -> 92.3 mm, vias 0 -> 4
- net /Input Phone Jacks/ptRX6: track 0.00 -> 92.3 mm, vias 0 -> 4
- net /Input Phone Jacks/ptRX8: track 0.00 -> 92.3 mm, vias 0 -> 4
- net /Input Phone Jacks/ptRX7: track 0.00 -> 92.3 mm, vias 0 -> 4
- net /Input Phone Jacks/ptRX20: track 0.00 -> 92.3 mm, vias 0 -> 4
- net /Input Phone Jacks/ptRX17: track 0.00 -> 92.3 mm, vias 0 -> 4
- net /Input Phone Jacks/ptRX15: track 0.00 -> 92.3 mm, vias 0 -> 4
- net /Input Phone Jacks/ptRX12: track 0.00 -> 92.3 mm, vias 0 -> 4
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
Commit message: holy crap trace routing speedrun
Parts:
- moved R1 332.0 mm to (752.6, 234.0)
- moved R102 329.0 mm to (752.6, 242.0)
- moved R103 326.0 mm to (752.6, 250.0)
- moved J50 325.6 mm to (767.2, 239.3)
- moved R104 323.0 mm to (752.6, 258.0)
- moved R105 320.1 mm to (752.6, 266.0)
- moved R106 317.1 mm to (752.6, 274.0)
- moved J51 316.5 mm to (767.2, 247.3)
- moved U2 316.3 mm to (731.0, 255.9)
- moved J53 315.9 mm to (767.2, 263.3)
- moved R107 314.2 mm to (752.6, 282.0)
- moved R108 311.3 mm to (752.6, 290.0)
- moved R109 308.4 mm to (752.6, 298.0)
- moved J52 307.4 mm to (767.2, 255.3)
- moved J54 306.9 mm to (767.2, 271.3)
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Connections:
- K10 pad 3: unconnected-(K10-Pad3) -> Net-(JP30-B)
- K10 pad 4: /Input Phone Jacks/Line Control3/Tpbx -> Net-(JP30-A)
- K12 pad 3: unconnected-(K12-Pad3) -> Net-(JP31-B)
- K12 pad 4: /Input Phone Jacks/Line Control4/Tpbx -> Net-(JP31-A)
- K14 pad 3: unconnected-(K14-Pad3) -> Net-(JP32-B)
- K14 pad 4: /Input Phone Jacks/Line Control5/Tpbx -> Net-(JP32-A)
- K16 pad 3: unconnected-(K16-Pad3) -> Net-(JP33-B)
- K16 pad 4: /Input Phone Jacks/Line Control6/Tpbx -> Net-(JP33-A)
- K18 pad 3: unconnected-(K18-Pad3) -> Net-(JP34-B)
- K18 pad 4: /Input Phone Jacks/Line Control7/Tpbx -> Net-(JP34-A)
- K20 pad 3: unconnected-(K20-Pad3) -> Net-(JP35-B)
- K20 pad 4: /Input Phone Jacks/Line Control8/Tpbx -> Net-(JP35-A)
- K22 pad 3: unconnected-(K22-Pad3) -> Net-(JP36-B)
- K22 pad 4: /Input Phone Jacks/Line Control9/Tpbx -> Net-(JP36-A)
- K24 pad 3: unconnected-(K24-Pad3) -> Net-(JP37-B)
- K24 pad 4: /Input Phone Jacks/Line Control10/Tpbx -> Net-(JP37-A)
- K26 pad 3: unconnected-(K26-Pad3) -> Net-(JP38-B)
- K26 pad 4: /Input Phone Jacks/Line Control11/Tpbx -> Net-(JP38-A)
- K28 pad 3: unconnected-(K28-Pad3) -> Net-(JP39-B)
- K28 pad 4: /Input Phone Jacks/Line Control12/Tpbx -> Net-(JP39-A)
- K30 pad 3: unconnected-(K30-Pad3) -> Net-(JP40-B)
- K30 pad 4: /Input Phone Jacks/Line Control13/Tpbx -> Net-(JP40-A)
- K32 pad 3: unconnected-(K32-Pad3) -> Net-(JP41-B)
- K32 pad 4: /Input Phone Jacks/Line Control14/Tpbx -> Net-(JP41-A)
- K34 pad 3: unconnected-(K34-Pad3) -> Net-(JP42-B)
- K34 pad 4: /Input Phone Jacks/Line Control15/Tpbx -> Net-(JP42-A)
- K36 pad 3: unconnected-(K36-Pad3) -> Net-(JP43-B)
- K36 pad 4: /Input Phone Jacks/Line Control16/Tpbx -> Net-(JP43-A)
- K38 pad 3: unconnected-(K38-Pad3) -> Net-(JP44-B)
- K38 pad 4: /Input Phone Jacks/Line Control17/Tpbx -> Net-(JP44-A)
- K4 pad 3: unconnected-(K4-Pad3) -> Net-(JP27-B)
- K4 pad 4: /Input Phone Jacks/Line Control0/Tpbx -> Net-(JP27-A)
- K40 pad 3: unconnected-(K40-Pad3) -> Net-(JP45-B)
- K40 pad 4: /Input Phone Jacks/Line Control18/Tpbx -> Net-(JP45-A)
- K42 pad 3: unconnected-(K42-Pad3) -> Net-(JP46-B)
- K42 pad 4: /Input Phone Jacks/Line Control19/Tpbx -> Net-(JP46-A)
- K44 pad 3: unconnected-(K44-Pad3) -> Net-(JP47-B)
- K44 pad 4: /Input Phone Jacks/Line Control20/Tpbx -> Net-(JP47-A)
- K46 pad 3: unconnected-(K46-Pad3) -> Net-(JP48-B)
- K46 pad 4: /Input Phone Jacks/Line Control21/Tpbx -> Net-(JP48-A)
- K48 pad 3: unconnected-(K48-Pad3) -> Net-(JP49-B)
- K48 pad 4: /Input Phone Jacks/Line Control22/Tpbx -> Net-(JP49-A)
- K50 pad 3: unconnected-(K50-Pad3) -> Net-(JP50-B)
- K50 pad 4: /Input Phone Jacks/Line Control23/Tpbx -> Net-(JP50-A)
- K6 pad 3: unconnected-(K6-Pad3) -> Net-(JP28-B)
- K6 pad 4: /Input Phone Jacks/Line Control1/Tpbx -> Net-(JP28-A)
- K8 pad 3: unconnected-(K8-Pad3) -> Net-(JP29-B)
- K8 pad 4: /Input Phone Jacks/Line Control2/Tpbx -> Net-(JP29-A)
- Q10 pad 2: controlSW3 -> /Multiplexers/LineControl3
- Q11 pad 2: /hookSW4 -> hookSW4
- Q12 pad 2: controlSW4 -> /Multiplexers/LineControl4
- Q13 pad 2: /hookSW5 -> hookSW5
- Q14 pad 2: controlSW5 -> /Multiplexers/LineControl5
- Q15 pad 2: /hookSW6 -> hookSW6
- Q16 pad 2: controlSW6 -> /Multiplexers/LineControl6
- Q17 pad 2: /hookSW7 -> hookSW7
- Q18 pad 2: controlSW7 -> /Multiplexers/LineControl7
- Q19 pad 2: /hookSW8 -> hookSW8
- Q20 pad 2: controlSW8 -> /Multiplexers/LineControl8
- Q21 pad 2: /hookSW9 -> hookSW9
- Q22 pad 2: controlSW9 -> /Multiplexers/LineControl9
- Q23 pad 2: /hookSW10 -> hookSW10
- Q24 pad 2: controlSW10 -> /Multiplexers/LineControl10
- Q25 pad 2: /hookSW11 -> hookSW11
- Q26 pad 2: controlSW11 -> /Multiplexers/LineControl11
- Q27 pad 2: /hookSW12 -> hookSW12
- Q28 pad 2: controlSW12 -> /Multiplexers/LineControl12
- Q29 pad 2: /hookSW13 -> hookSW13
- Q3 pad 2: /hookSW0 -> hookSW0
- Q30 pad 2: controlSW13 -> /Multiplexers/LineControl13
- Q31 pad 2: /hookSW14 -> hookSW14
- Q32 pad 2: controlSW14 -> /Multiplexers/LineControl14
- Q33 pad 2: /hookSW15 -> hookSW15
- Q34 pad 2: controlSW15 -> /Multiplexers/LineControl15
- Q35 pad 2: /hookSW16 -> hookSW16
- Q36 pad 2: controlSW16 -> /Multiplexers/LineControl16
- Q37 pad 2: /hookSW17 -> hookSW17
- Q38 pad 2: controlSW17 -> /Multiplexers/LineControl17
- Q39 pad 2: /hookSW18 -> hookSW18
- Q4 pad 2: controlSW0 -> /Multiplexers/LineControl0
- Q40 pad 2: controlSW18 -> /Multiplexers/LineControl18
- Q41 pad 2: /hookSW19 -> hookSW19
- Q42 pad 2: controlSW19 -> /Multiplexers/LineControl19
- Q43 pad 2: /hookSW20 -> hookSW20
- Q44 pad 2: controlSW20 -> /Multiplexers/LineControl20
- Q45 pad 2: /hookSW21 -> hookSW21
- Q46 pad 2: controlSW21 -> /Multiplexers/LineControl21
- Q47 pad 2: /hookSW22 -> hookSW22
- Q48 pad 2: controlSW22 -> /Multiplexers/LineControl22
- Q49 pad 2: /hookSW23 -> hookSW23
- Q5 pad 2: /hookSW1 -> hookSW1
- Q50 pad 2: controlSW23 -> /Multiplexers/LineControl23
- Q6 pad 2: controlSW1 -> /Multiplexers/LineControl1
- Q7 pad 2: /hookSW2 -> hookSW2
- Q8 pad 2: controlSW2 -> /Multiplexers/LineControl2
- Q9 pad 2: /hookSW3 -> hookSW3
- R11 pad 1: controlSW1 -> /Multiplexers/LineControl1
- R12 pad 2: /hookSW2 -> hookSW2
- R14 pad 1: controlSW2 -> /Multiplexers/LineControl2
- R15 pad 2: /hookSW3 -> hookSW3
- R17 pad 1: controlSW3 -> /Multiplexers/LineControl3
- R18 pad 2: /hookSW4 -> hookSW4
- R20 pad 1: controlSW4 -> /Multiplexers/LineControl4
- R21 pad 2: /hookSW5 -> hookSW5
- R23 pad 1: controlSW5 -> /Multiplexers/LineControl5
- R24 pad 2: /hookSW6 -> hookSW6
- R26 pad 1: controlSW6 -> /Multiplexers/LineControl6
- R27 pad 2: /hookSW7 -> hookSW7
- R29 pad 1: controlSW7 -> /Multiplexers/LineControl7
- R30 pad 2: /hookSW8 -> hookSW8
- R32 pad 1: controlSW8 -> /Multiplexers/LineControl8
- R33 pad 2: /hookSW9 -> hookSW9
- R35 pad 1: controlSW9 -> /Multiplexers/LineControl9
- R36 pad 2: /hookSW10 -> hookSW10
- R38 pad 1: controlSW10 -> /Multiplexers/LineControl10
- R39 pad 2: /hookSW11 -> hookSW11
- R41 pad 1: controlSW11 -> /Multiplexers/LineControl11
- R42 pad 2: /hookSW12 -> hookSW12
- R44 pad 1: controlSW12 -> /Multiplexers/LineControl12
- R45 pad 2: /hookSW13 -> hookSW13
- R47 pad 1: controlSW13 -> /Multiplexers/LineControl13
- R48 pad 2: /hookSW14 -> hookSW14
- R50 pad 1: controlSW14 -> /Multiplexers/LineControl14
- R51 pad 2: /hookSW15 -> hookSW15
- R53 pad 1: controlSW15 -> /Multiplexers/LineControl15
- R54 pad 2: /hookSW16 -> hookSW16
- R56 pad 1: controlSW16 -> /Multiplexers/LineControl16
- R57 pad 2: /hookSW17 -> hookSW17
- R59 pad 1: controlSW17 -> /Multiplexers/LineControl17
- R6 pad 2: /hookSW0 -> hookSW0
- R60 pad 2: /hookSW18 -> hookSW18
- R62 pad 1: controlSW18 -> /Multiplexers/LineControl18
- R63 pad 2: /hookSW19 -> hookSW19
- R65 pad 1: controlSW19 -> /Multiplexers/LineControl19
- R66 pad 2: /hookSW20 -> hookSW20
- R68 pad 1: controlSW20 -> /Multiplexers/LineControl20
- R69 pad 2: /hookSW21 -> hookSW21
- R71 pad 1: controlSW21 -> /Multiplexers/LineControl21
- R72 pad 2: /hookSW22 -> hookSW22
- R74 pad 1: controlSW22 -> /Multiplexers/LineControl22
- R75 pad 2: /hookSW23 -> hookSW23
- R77 pad 1: controlSW23 -> /Multiplexers/LineControl23
- R8 pad 1: controlSW0 -> /Multiplexers/LineControl0
- R9 pad 2: /hookSW1 -> hookSW1
- U1 pad 19: GND -> GNDD
- U1 pad 20: GND -> GNDD
- U1 pad 22: GND -> GNDD
- U1 pad 32: controlSW23 -> hookSW23
- U1 pad 34: controlSW22 -> hookSW22
- U1 pad 35: controlSW21 -> hookSW21
- U1 pad 36: controlSW20 -> hookSW20
- U1 pad 37: controlSW19 -> hookSW19
- U1 pad 38: controlSW18 -> hookSW18
- U1 pad 49: GND -> GNDD
- U1 pad 57: controlSW0 -> hookSW0
- U1 pad 58: controlSW1 -> hookSW1
- U1 pad 59: controlSW2 -> hookSW2
- U1 pad 60: GND -> GNDD
- U1 pad 61: controlSW3 -> hookSW3
- U1 pad 62: controlSW4 -> hookSW4
- U1 pad 63: controlSW5 -> hookSW5
- U1 pad 64: controlSW6 -> hookSW6
- U1 pad 65: controlSW7 -> hookSW7
- U1 pad 66: controlSW8 -> hookSW8
- U1 pad 67: controlSW9 -> hookSW9
- U1 pad 68: controlSW10 -> hookSW10
- U1 pad 69: controlSW11 -> hookSW11
- U1 pad 70: controlSW12 -> hookSW12
- U1 pad 71: controlSW13 -> hookSW13
- U1 pad 72: GND -> GNDD
- U1 pad 73: controlSW14 -> hookSW14
- U1 pad 74: controlSW15 -> hookSW15
- U1 pad 75: controlSW16 -> hookSW16
- U1 pad 77: controlSW17 -> hookSW17
- U1 pad 8: GND -> GNDD
- U4 pad 8: /Multiplexers/Vss -> GNDD
- U5 pad 4: /Multiplexers/Vss -> GNDD
- U5 pad 8: /Multiplexers/Vss -> GNDD
- U6 pad 5: /Multiplexers/Vss -> GNDD
- U6 pad 8: /Multiplexers/Vss -> GNDD
- U7 pad 14: /ADC/AGND -> GNDD
- U7 pad 9: /ADC/DGND -> GNDD
- U8 pad 14: /ADC/AGND -> GNDD
- U8 pad 9: /ADC/DGND -> GNDD
- U9 pad 14: /ADC/AGND -> GNDD
- U9 pad 9: /ADC/DGND -> GNDD
Routing:
- net shiftLd: track 0.00 -> 840.0 mm, vias 0 -> 1
- net shiftClk: track 0.00 -> 833.7 mm, vias 0 -> 2
- net shiftInh: track 0.00 -> 773.5 mm, vias 0 -> 2
- net shiftOut: track 0.00 -> 768.1 mm
- net /ADC/ADC23: track 86.0 -> 678.2 mm, vias 0 -> 1
- net /ADC/ADC22: track 80.4 -> 668.3 mm, vias 0 -> 1
- net /ADC/ADC19: track 28.9 -> 605.1 mm, vias 0 -> 1
- net /ADC/ADC21: track 76.3 -> 647.2 mm, vias 0 -> 1
- net /ADC/ADC20: track 77.5 -> 627.2 mm, vias 0 -> 1
- net /ADC/ADC18: track 28.9 -> 575.1 mm, vias 0 -> 1
- net /ADC/ADC17: track 28.9 -> 548.8 mm
- net /ADC/ADC16: track 28.9 -> 527.9 mm, vias 0 -> 1
- net /ADC/ADC15: track 28.9 -> 503.3 mm, vias 0 -> 1
- net /ADC/ADC14: track 28.9 -> 483.3 mm, vias 0 -> 1
- net /ADC/ADC13: track 28.9 -> 463.4 mm, vias 0 -> 1
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Other:
- board text removed: "Input Jacks"
- board text removed: "Output Jacks"
