File: kicad/pbx-sniffer/merge sniffer.kicad_pcb (KiCad board)
At the start: 2 copper layers, 343 parts, among them K10 Relay_SPDT, K11 Relay_SPST-NO, K12 Relay_SPDT, K13 Relay_SPST-NO, K14 Relay_SPDT, K15 Relay_SPST-NO, K16 Relay_SPDT, K17 Relay_SPST-NO, K18 Relay_SPDT, K19 Relay_SPST-NO, K20 Relay_SPDT, K21 Relay_SPST-NO, K22 Relay_SPDT, K23 Relay_SPST-NO, K24 Relay_SPDT, K25 Relay_SPST-NO, K26 Relay_SPDT, K27 Relay_SPST-NO, K28 Relay_SPDT, K29 Relay_SPST-NO, K3 Relay_SPST-NO, K30 Relay_SPDT, K31 Relay_SPST-NO, K32 Relay_SPDT, K33 Relay_SPST-NO, K34 Relay_SPDT, K35 Relay_SPST-NO, K36 Relay_SPDT, K37 Relay_SPST-NO, K38 Relay_SPDT, K39 Relay_SPST-NO, K4 Relay_SPDT, K40 Relay_SPDT, K41 Relay_SPST-NO, K42 Relay_SPDT, K43 Relay_SPST-NO, K44 Relay_SPDT, K45 Relay_SPST-NO, K46 Relay_SPDT, K47 Relay_SPST-NO, K48 Relay_SPDT, K49 Relay_SPST-NO, K5 Relay_SPST-NO, K50 Relay_SPDT, K6 Relay_SPDT, K7 Relay_SPST-NO, K8 Relay_SPDT, K9 Relay_SPST-NO, Q10 PMOS, Q11 PMOS, Q12 PMOS, Q13 PMOS, Q14 PMOS, Q15 PMOS, Q16 PMOS, Q17 PMOS, Q18 PMOS, Q19 PMOS, Q20 PMOS, Q21 PMOS, Q22 PMOS, Q23 PMOS, Q24 PMOS, Q25 PMOS, Q26 PMOS, Q27 PMOS, Q28 PMOS, Q29 PMOS, Q3 PMOS, Q30 PMOS, Q31 PMOS, Q32 PMOS, Q33 PMOS, Q34 PMOS, Q35 PMOS, Q36 PMOS, Q37 PMOS, Q38 PMOS, Q39 PMOS, Q4 PMOS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

Commit message: mostly finished wiring one column
Routing:
- net /Input Phone Jacks/ptRX16: track 297.4 -> 0.00 mm, vias 2 -> 0
- net /Input Phone Jacks/Rpbx16: track 297.4 -> 0.00 mm, vias 3 -> 0
- net /Input Phone Jacks/ptRX8: track 249.0 -> 0.00 mm, vias 2 -> 0
- net /Input Phone Jacks/Rpbx8: track 249.0 -> 0.00 mm, vias 3 -> 0
- net /Input Phone Jacks/ptRX0: track 198.7 -> 0.00 mm, vias 2 -> 0
- net /Input Phone Jacks/Line Control16/Tpbx: track 173.6 -> 95.7 mm
- net /Input Phone Jacks/Line Control8/Tpbx: track 123.0 -> 51.1 mm
- net /Input Phone Jacks/Line Control0/Tpbx: track 76.4 -> 14.3 mm
- net /Input Phone Jacks/Rpbx0: track 18.2 -> 0.00 mm, vias 1 -> 0
- removed copper zone on B.Cu, net +5V
- removed copper zone on F.Cu, net GNDD
