File: kicad/pbx-sniffer/tobe-wc.kicad_pcb (KiCad board)
At the start: 2 copper layers, 377 parts, among them J49 Conn_01x02_Socket, J50 Conn_01x02_Socket, J51 Conn_01x02_Socket, J52 Conn_01x02_Socket, J53 Conn_01x02_Socket, J54 Conn_01x02_Socket, J55 Conn_01x02_Socket, J56 Conn_01x02_Socket, J57 Conn_01x02_Socket, J58 Conn_01x02_Socket, J59 Conn_01x02_Socket, J60 Conn_01x02_Socket, J61 Conn_01x02_Socket, J62 Conn_01x02_Socket, J63 Conn_01x02_Socket, J64 Conn_01x02_Socket, K10 Relay_SPDT, K11 Relay_SPST-NO, K12 Relay_SPDT, K13 Relay_SPST-NO, K14 Relay_SPDT, K15 Relay_SPST-NO, K16 Relay_SPDT, K17 Relay_SPST-NO, K18 Relay_SPDT, K19 Relay_SPST-NO, K20 Relay_SPDT, K21 Relay_SPST-NO, K22 Relay_SPDT, K23 Relay_SPST-NO, K24 Relay_SPDT, K25 Relay_SPST-NO, K26 Relay_SPDT, K27 Relay_SPST-NO, K28 Relay_SPDT, K29 Relay_SPST-NO, K3 Relay_SPST-NO, K30 Relay_SPDT, K31 Relay_SPST-NO, K32 Relay_SPDT, K33 Relay_SPST-NO, K34 Relay_SPDT, K35 Relay_SPST-NO, K36 Relay_SPDT, K37 Relay_SPST-NO, K38 Relay_SPDT, K39 Relay_SPST-NO, K4 Relay_SPDT, K40 Relay_SPDT, K41 Relay_SPST-NO, K42 Relay_SPDT, K43 Relay_SPST-NO, K44 Relay_SPDT, K45 Relay_SPST-NO, K46 Relay_SPDT, K47 Relay_SPST-NO, K48 Relay_SPDT, K49 Relay_SPST-NO, K5 Relay_SPST-NO, K50 Relay_SPDT, K6 Relay_SPDT, K7 Relay_SPST-NO, K8 Relay_SPDT, K9 Relay_SPST-NO, Q10 PMOS, Q11 PMOS, Q12 PMOS, Q13 PMOS, Q14 PMOS, Q15 PMOS, Q16 PMOS, Q17 PMOS, Q18 PMOS, Q19 PMOS, Q20 PMOS, Q21 PMOS, Q22 PMOS, Q23 PMOS, Q24 PMOS, Q25 PMOS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

Commit message: holy crap trace routing speedrun
Parts:
- moved J64 68.5 mm to (552.4, 367.3)
- moved J63 61.1 mm to (552.4, 359.3)
- moved J62 54.1 mm to (552.4, 351.3)
- moved J61 47.9 mm to (552.4, 343.3)
- moved J60 43.8 mm to (552.4, 335.3)
- moved U2 38.1 mm to (516.2, 271.9)
- moved J59 36.6 mm to (552.4, 327.3)
- moved R116 36.6 mm to (537.8, 370.0)
- moved J49 35.1 mm to (552.4, 247.3)
- moved R115 33.2 mm to (537.8, 362.0)
- moved U34 32.9 mm to (516.2, 322.6)
- moved R1 32.3 mm to (537.8, 250.0)
- moved J58 30.7 mm to (552.4, 319.3)
- moved R114 29.9 mm to (537.8, 354.0)
- moved R102 29.1 mm to (537.8, 258.0)
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Routing:
- net +5V: track 0.00 -> 332.9 mm, vias 0 -> 2
- net /Shift Registers/TBTN0: track 0.00 -> 59.2 mm
- net /Shift Registers/TBTN9: track 0.00 -> 55.3 mm, vias 0 -> 1
- net /Shift Registers/TBTN3: track 0.00 -> 54.1 mm, vias 0 -> 1
- net /Shift Registers/TBTN10: track 0.00 -> 54.1 mm, vias 0 -> 1
- net /Shift Registers/TBTN15: track 0.00 -> 52.4 mm
- net /Shift Registers/TBTN11: track 0.00 -> 51.6 mm
- net /Shift Registers/TBTN1: track 0.00 -> 50.8 mm, vias 0 -> 1
- net /Shift Registers/TBTN7: track 0.00 -> 44.0 mm, vias 0 -> 1
- net /Shift Registers/TBTN8: track 0.00 -> 43.6 mm
- net /Shift Registers/TBTN2: track 0.00 -> 43.0 mm, vias 0 -> 1
- net /Shift Registers/TBTN6: track 0.00 -> 41.0 mm, vias 0 -> 1
- net /Shift Registers/TBTN14: track 0.00 -> 34.2 mm
- net /Shift Registers/TBTN12: track 0.00 -> 34.0 mm, vias 0 -> 1
- net /Shift Registers/TBTN4: track 0.00 -> 33.7 mm, vias 0 -> 1
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