File: kicad/pbx-sniffer/adc.kicad_sch (KiCad schematic)
At the start: 0 parts

Commit message: updated multiplexer with busses, added ADCs, fixed relay sch
Parts:
- added U10, U8, U9: MCP3008, Package_DIP:DIP-16_W7.62mm, symbol Analog_ADC:MCP3008
Connections:
- new net ADC0: U8.1 (CH0)
- new net ADC1: U8.2 (CH1)
- new net ADC10: U9.3 (CH2)
- new net ADC11: U9.4 (CH3)
- new net ADC12: U9.5 (CH4)
- new net ADC13: U9.6 (CH5)
- new net ADC14: U9.7 (CH6)
- new net ADC15: U9.8 (CH7)
- new net ADC16: U10.1 (CH0)
- new net ADC17: U10.2 (CH1)
- new net ADC18: U10.3 (CH2)
- new net ADC19: U10.4 (CH3)
- new net ADC2: U8.3 (CH2)
- new net ADC20: U10.5 (CH4)
- new net ADC21: U10.6 (CH5)
- new net ADC22: U10.7 (CH6)
- new net ADC23: U10.8 (CH7)
- new net ADC3: U8.4 (CH3)
- new net ADC4: U8.5 (CH4)
- new net ADC5: U8.6 (CH5)
- new net ADC6: U8.7 (CH6)
- new net ADC7: U8.8 (CH7)
- new net ADC8: U9.1 (CH0)
- new net ADC9: U9.2 (CH1)
- new net ADCclk: U10.13 (CLK), U8.13 (CLK), U9.13 (CLK)
- new net ADCrx: U10.11 (Din), U8.11 (Din), U9.11 (Din)
- new net ADCs0: U8.10 (~{CS}/SHDN)
- new net ADCs1: U9.10 (~{CS}/SHDN)
- new net ADCs2: U10.10 (~{CS}/SHDN)
- new net ADCtx: U10.12 (Dout), U8.12 (Dout), U9.12 (Dout)
- new net AGND: U10.14 (AGND), U8.14 (AGND), U9.14 (AGND)
- new net DGND: U10.9 (DGND), U8.9 (DGND), U9.9 (DGND)
- new net Vdd: U10.16 (Vdd), U8.16 (Vdd), U9.16 (Vdd)
- new net Vref: U10.15 (Vref), U8.15 (Vref), U9.15 (Vref)

Commit message: commenced placement on pcb
Parts:
- renumbered U8 to U7, U9 to U8, U10 to U9
Changed lines of the file:
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@@
 		(on_board yes)
 		(dnp no)
-		(property "Reference" "U10"
+		(property "Reference" "U9"
 			(at 108.585 116.84 0)
 			(effects
@@
 			(project "pbx-sniffer"
 				(path "/4a5b9b8a-323a-4796-bf73-ccba532d2e31/034ac82b-541e-40fe-babd-660f127c9f12"
-					(reference "U10")
+					(reference "U9")
 					(unit 1)
 				)
@@
 		(on_board yes)
 		(dnp no)
-		(property "Reference" "U9"
+		(property "Reference" "U8"
 			(at 108.585 73.66 0)
 			(effects
@@
 			(project "pbx-sniffer"
 				(path "/4a5b9b8a-323a-4796-bf73-ccba532d2e31/034ac82b-541e-40fe-babd-660f127c9f12"
-					(reference "U9")
+					(reference "U8")
 					(unit 1)
 				)
@@
 		(on_board yes)
 		(dnp no)
-		(property "Reference" "U8"
+		(property "Reference" "U7"
 			(at 108.585 27.94 0)
 			(effects
@@
 			(project ""
 				(path "/4a5b9b8a-323a-4796-bf73-ccba532d2e31/034ac82b-541e-40fe-babd-660f127c9f12"
-					(reference "U8")
+					(reference "U7")
 					(unit 1)
 				)

Commit message: add part numbers for remaining important parts
Parts:
- U7, U8, U9: DKPN (none) -> MCP3008-I/P-ND
Changed lines of the file:
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@@
+			)
+		)
+		(property "DKPN" "MCP3008-I/P-ND"
+			(at 116.84 131.445 0)
+			(effects
+				(font
+					(size 1.27 1.27)
+				)
+				(hide yes)
 			)
 		)
@@
 			)
 		)
+		(property "DKPN" "MCP3008-I/P-ND"
+			(at 116.84 88.265 0)
+			(effects
+				(font
+					(size 1.27 1.27)
+				)
+				(hide yes)
+			)
+		)
 		(pin "10"
 		)
@@
 			(at 116.84 42.545 0)
 			(effects
+				(font
+					(size 1.27 1.27)
+				)
+				(hide yes)
+			)
+		)
+		(property "DKPN" "MCP3008-I/P-ND"
+			(at 116.84 42.545 0)
+			(effects
