File: kicad/pbx-sniffer/relays.kicad_sch (KiCad schematic)
At the start: 9 parts, among them K1 Relay_SPST-NO, K2 Relay_SPDT, Q1 PMOS, Q2 PMOS

Commit message: add part numbers for remaining important parts
Parts:
- D2, D3: DKPN (none) -> 2368-1N4003-ND
- K1: DKPN (none) -> 1835-1116-ND
- K2: DKPN (none) -> 3385-AZ943-1CH-5DE-ND
- Q1, Q2: DKPN (none) -> ZVP3306A-ND
Changed lines of the file:
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@@
+			)
+		)
+		(property "DKPN" "3385-AZ943-1CH-5DE-ND"
+			(at 104.902 45.72 90)
+			(effects
+				(font
+					(size 1.27 1.27)
+				)
+				(hide yes)
 			)
 		)
@@
 			)
 		)
+		(property "DKPN" "2368-1N4003-ND"
+			(at 79.375 53.975 90)
+			(effects
+				(font
+					(size 1.27 1.27)
+				)
+				(hide yes)
+			)
+		)
 		(pin "1"
 		)
@@
 			)
 		)
+		(property "DKPN" "ZVP3306A-ND"
+			(at 67.945 41.275 0)
+			(effects
+				(font
+					(size 1.27 1.27)
+				)
+				(hide yes)
+			)
+		)
 		(pin "3"
 		)
@@
 		)
 		(property "Sim.Pins" "1=K 2=A"
+			(at 104.394 59.182 0)
+			(effects
+				(font
+					(size 1.27 1.27)
+				)
+				(hide yes)
+			)
+		)
+		(property "DKPN" "2368-1N4003-ND"
 			(at 104.394 59.182 0)
 			(effects
@@
 			)
 		)
+		(property "DKPN" "1835-1116-ND"
+			(at 65.405 53.975 0)
+			(effects
+				(font
+					(size 1.27 1.27)
+				)
+				(hide yes)
+			)
+		)
 		(pin "5"
 		)
@@
 			(effects
 				(font
+					(size 1.27 1.27)
+				)
+				(hide yes)
+			)
+		)
+		(property "DKPN" "ZVP3306A-ND"
+			(at 91.44 56.388 0)
+			(effects
+				(font

Commit message: module modularized
Parts:
- added JP26: Jumper_3_Bridged12, symbol Jumper:Jumper_3_Bridged12
Connections:
- net Tpbx: now also JP26.2 (C); no longer K2.4
- net at K2.3: now also JP26.3 (B)
- new net: JP26.1 (A), K2.4
Other:
- moved on the sheet: K2
Changed lines of the file:
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@@
+	)
+	(junction
+		(at 82.55 36.83)
+		(diameter 0)
+		(color 0 0 0 0)
 	)
 	(junction
@@
 	(wire
 		(pts
-			(xy 97.282 53.848) (xy 97.282 50.8)
+			(xy 97.282 53.848) (xy 97.79 50.8)
 		)
 		(stroke
@@
 	(wire
 		(pts
-			(xy 60.325 30.48) (xy 85.725 30.48)
+			(xy 60.325 30.48) (xy 82.55 30.48)
 		)
 		(stroke
@@
 	(wire
 		(pts
-			(xy 112.522 40.64) (xy 120.65 40.64)
+			(xy 113.03 40.64) (xy 120.65 40.64)
 		)
 		(stroke
@@
 	(wire
 		(pts
-			(xy 85.725 43.18) (xy 97.282 43.18)
-		)
-		(stroke
-			(width 0)
-			(type default)
-		)
-	)
-	(wire
-		(pts
 			(xy 83.312 71.882) (xy 83.312 71.12)
 		)
@@
 	(wire
 		(pts
+			(xy 86.36 43.18) (xy 97.79 43.18)
+		)
+		(stroke
+			(width 0)
+			(type default)
+		)
+	)
+	(wire
+		(pts
 			(xy 79.375 46.355) (xy 70.485 46.355)
 		)
@@
 	(wire
 		(pts
+			(xy 82.55 36.83) (xy 82.55 43.18)
+		)
+		(stroke
+			(width 0)
+			(type default)
+		)
+	)
+	(wire
+		(pts
 			(xy 118.618 58.928) (xy 118.618 59.182)
 		)
@@
 	(wire
 		(pts
+			(xy 97.79 30.48) (xy 86.36 30.48)
+		)
+		(stroke
+			(width 0)
+			(type default)
+		)
+	)
+	(wire
+		(pts
 			(xy 43.815 30.48) (xy 60.325 30.48)
 		)
@@
 	(wire
 		(pts
-			(xy 118.364 50.8) (xy 112.522 50.8)
+			(xy 118.364 50.8) (xy 113.03 50.8)
 		)
 		(stroke
@@
 	(wire
 		(pts
+			(xy 97.79 38.1) (xy 97.79 30.48)
+		)
+		(stroke
+			(width 0)
+			(type default)
+		)
+	)
+	(wire
+		(pts
 			(xy 118.618 58.928) (xy 118.872 58.928)
 		)
@@
 	(wire
 		(pts
-			(xy 85.725 30.48) (xy 85.725 43.18)
+			(xy 82.55 30.48) (xy 82.55 36.83)
 		)
 		(stroke
@@
 			)
 			(justify right)
+		)
+	)
+	(symbol
+		(lib_id "Jumper:Jumper_3_Bridged12")
+		(at 86.36 36.83 270)
+		(mirror x)
+		(unit 1)
+		(exclude_from_sim no)
+		(in_bom no)
+		(on_board yes)
+		(dnp no)
+		(property "Reference" "JP26"
+			(at 88.9 38.1001 90)
+			(effects
+				(font
+					(size 1.27 1.27)
+				)
+				(justify left)
+			)
+		)
+		(property "Value" "Jumper_3_Bridged12"
+			(at 88.9 35.5601 90)
+			(effects
+				(font
+					(size 1.27 1.27)
+				)
+				(justify left)
+			)
+		)
+		(property "Footprint" ""
+			(at 86.36 36.83 0)
+			(effects
+				(font
+					(size 1.27 1.27)
+				)
+				(hide yes)
+			)
+		)
+		(property "Datasheet" "~"
+			(at 86.36 36.83 0)
+			(effects
+				(font
+					(size 1.27 1.27)
+				)
+				(hide yes)
+			)
+		)
+		(property "Description" "Jumper, 3-pole, pins 1+2 closed/bridged"
+			(at 86.36 36.83 0)
+			(effects
+				(font
+					(size 1.27 1.27)
+				)
+				(hide yes)
+			)
+		)
+		(pin "3"
+		)
+		(pin "2"
+		)
+		(pin "1"
+		)
+		(instances
+			(project ""
+				(path "/4a5b9b8a-323a-4796-bf73-ccba532d2e31/992e173b-e387-457c-8c0b-8a825a1cd866"
+					(reference "JP26")
+					(unit 1)
+				)
+				(path "/4a5b9b8a-323a-4796-bf73-ccba532d2e31/7f66e062-f194-4d68-9744-df7dfe6719d2/00f56bf1-07c3-4f46-80f2-1ee35ffc2d93"
+					(reference "JP41")
+					(unit 1)
+				)
+				(path "/4a5b9b8a-323a-4796-bf73-ccba532d2e31/7f66e062-f194-4d68-9744-df7dfe6719d2/1eb0fa64-96ac-44d0-814e-84824698e86b"
+					(reference "JP35")
+					(unit 1)
+				)
+				(path "/4a5b9b8a-323a-4796-bf73-ccba532d2e31/7f66e062-f194-4d68-9744-df7dfe6719d2/38816e2a-7a2b-4973-bcec-df3663d4cf5f"
+					(reference "JP30")
+					(unit 1)
+				)
+				(path "/4a5b9b8a-323a-4796-bf73-ccba532d2e31/7f66e062-f194-4d68-9744-df7dfe6719d2/42a11760-5991-4a27-bb66-96affc9cf5be"
+					(reference "JP44")
+					(unit 1)
+				)
+				(path "/4a5b9b8a-323a-4796-bf73-ccba532d2e31/7f66e062-f194-4d68-9744-df7dfe6719d2/44ad5056-482d-4f8d-bb50-3e43cf948a11"
+					(reference "JP40")
+					(unit 1)
+				)
+				(path "/4a5b9b8a-323a-4796-bf73-ccba532d2e31/7f66e062-f194-4d68-9744-df7dfe6719d2/773cd5d7-4854-4731-b793-55c612d84e2a"
+					(reference "JP50")
+					(unit 1)
+				)
+				(path "/4a5b9b8a-323a-4796-bf73-ccba532d2e31/7f66e062-f194-4d68-9744-df7dfe6719d2/79e3cd55-6732-4d3b-a542-29154c7f464f"
+					(reference "JP29")
+					(unit 1)
+				)
+				(path "/4a5b9b8a-323a-4796-bf73-ccba532d2e31/7f66e062-f194-4d68-9744-df7dfe6719d2/8d49db71-2d1c-4772-8b54-83322075e384"
+					(reference "JP34")
+					(unit 1)
+				)
+				(path "/4a5b9b8a-323a-4796-bf73-ccba532d2e31/7f66e062-f194-4d68-9744-df7dfe6719d2/8d655c60-c0bf-4622-a513-3bbb77027fd7"
+					(reference "JP46")
+					(unit 1)
+				)
+				(path "/4a5b9b8a-323a-4796-bf73-ccba532d2e31/7f66e062-f194-4d68-9744-df7dfe6719d2/8ee9859b-1672-4437-94a5-3c272c0a6aea"
+					(reference "JP31")
+					(unit 1)
+				)
+				(path "/4a5b9b8a-323a-4796-bf73-ccba532d2e31/7f66e062-f194-4d68-9744-df7dfe6719d2/916f6c44-6f38-4b22-b3b2-119000030de9"
+					(reference "JP42")
+					(unit 1)
+				)
+				(path "/4a5b9b8a-323a-4796-bf73-ccba532d2e31/7f66e062-f194-4d68-9744-df7dfe6719d2/92ab2728-cc70-42ea-aa6d-c5c8e6aa9c07"
+					(reference "JP27")
+					(unit 1)
+				)
+				(path "/4a5b9b8a-323a-4796-bf73-ccba532d2e31/7f66e062-f194-4d68-9744-df7dfe6719d2/96becac7-5a0e-4930-90a4-44919452acb8"
+					(reference "JP28")
+					(unit 1)
+				)
+				(path "/4a5b9b8a-323a-4796-bf73-ccba532d2e31/7f66e062-f194-4d68-9744-df7dfe6719d2/98d66f06-d8c1-4ad8-971f-442fe3242d04"
+					(reference "JP33")
+					(unit 1)
+				)
+				(path "/4a5b9b8a-323a-4796-bf73-ccba532d2e31/7f66e062-f194-4d68-9744-df7dfe6719d2/9a250a20-5681-43c1-a486-9e70dc1b4814"
+					(reference "JP49")
+					(unit 1)
+				)
+				(path "/4a5b9b8a-323a-4796-bf73-ccba532d2e31/7f66e062-f194-4d68-9744-df7dfe6719d2/9c2d885a-5535-4c7e-8888-9f58e07d8fce"
+					(reference "JP47")
+					(unit 1)
+				)
+				(path "/4a5b9b8a-323a-4796-bf73-ccba532d2e31/7f66e062-f194-4d68-9744-df7dfe6719d2/a28bdb06-e675-4415-aab2-e7ceac7e199e"
+					(reference "JP48")
+					(unit 1)
+				)
+				(path "/4a5b9b8a-323a-4796-bf73-ccba532d2e31/7f66e062-f194-4d68-9744-df7dfe6719d2/b3e5c1a4-8db6-47cd-94ff-28875d6b5a9f"
+					(reference "JP43")
+					(unit 1)
+				)
+				(path "/4a5b9b8a-323a-4796-bf73-ccba532d2e31/7f66e062-f194-4d68-9744-df7dfe6719d2/da4ef1be-9554-46f7-930f-105f0924ad30"
+					(reference "JP45")
+					(unit 1)
+				)
+				(path "/4a5b9b8a-323a-4796-bf73-ccba532d2e31/7f66e062-f194-4d68-9744-df7dfe6719d2/e79f967e-b2ae-4ffb-a428-372046ccf89d"
+					(reference "JP32")
+					(unit 1)
+				)
+				(path "/4a5b9b8a-323a-4796-bf73-ccba532d2e31/7f66e062-f194-4d68-9744-df7dfe6719d2/eaece676-439e-4621-bcab-fd48f3494033"
+					(reference "JP39")
+					(unit 1)
+				)
+				(path "/4a5b9b8a-323a-4796-bf73-ccba532d2e31/7f66e062-f194-4d68-9744-df7dfe6719d2/ed188815-edb9-4844-b657-59d30b497536"
+					(reference "JP37")
+					(unit 1)
+				)
+				(path "/4a5b9b8a-323a-4796-bf73-ccba532d2e31/7f66e062-f194-4d68-9744-df7dfe6719d2/edb59804-8171-450e-bcbc-70b4ff57a57d"
+					(reference "JP38")
+					(unit 1)
+				)
+				(path "/4a5b9b8a-323a-4796-bf73-ccba532d2e31/7f66e062-f194-4d68-9744-df7dfe6719d2/f19706de-4a26-4420-8554-8f68cb4e294e"
+					(reference "JP36")
+					(unit 1)
+				)
+			)
 		)
 	)
@@
 	(symbol
 		(lib_id "Relay:Relay_SPDT")
-		(at 104.902 45.72 90)
+		(at 105.41 45.72 90)
 		(unit 1)
 		(exclude_from_sim no)
@@
 		(fields_autoplaced yes)
 		(property "Reference" "K2"
-			(at 104.902 31.115 90)
+			(at 105.41 31.115 90)
 			(effects
 				(font
@@
 		)
 		(property "Value" "Relay_SPDT"
-			(at 104.902 33.655 90)
+			(at 105.41 33.655 90)
 			(effects
 				(font
@@
 		)
 		(property "Footprint" "Phones:K_AZ943-1C_AMZ"
-			(at 106.172 34.29 0)
+			(at 106.68 34.29 0)
 			(effects
 				(font
@@
 		)
 		(property "Datasheet" "https://www.azettler.com/pdfs/az943.pdf"
-			(at 104.902 45.72 0)
+			(at 105.41 45.72 0)
 			(effects
 				(font
@@
 		)
 		(property "Description" "Relay SPDT, monostable, EN50005"
-			(at 104.902 45.72 0)
+			(at 105.41 45.72 0)
 			(effects
 				(font
@@
 		)
 		(property "DKPN" "3385-AZ943-1CH-5DE-ND"
-			(at 104.902 45.72 90)
-			(effects
-				(font
+			(at 105.41 45.72 90)
+			(effects
+				(font

Commit message: added solderjumpers for the control relays
Parts:
- JP26: footprint (none) -> Jumper:SolderJumper-3_P1.3mm_Bridged2Bar12_RoundedPad1.0x1.5mm
Changed lines of the file:
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@@
 			)
 		)
-		(property "Footprint" ""
+		(property "Footprint" "Jumper:SolderJumper-3_P1.3mm_Bridged2Bar12_RoundedPad1.0x1.5mm"
 			(at 86.36 36.83 0)
 			(effects
